File: Atari130KB/Atari130KB.kicad_pcb (KiCad board)
At the start: 2 copper layers, 64 parts

Commit message: Improve Ids of 130MX components
Parts:
- renumbered Conn_Main1 to Conn_Main, SW_*1 to SW_*, SW_+1 to SW_+, SW_,1 to SW_,, SW_-1 to SW_-, SW_.1 to SW_.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
