File: JoyKeyMX/AtariJoystickPaddleTester/AtariJoystickPaddleTester.kicad_sch (KiCad schematic)
At the start: 48 parts, among them J1 DB9_Male, J2 Barrel_Jack, SW1 SWITCH, U1 LM7809_TO220, U2 LM3914V, U3 LM3914V

Commit message: Change switch footprint
Parts:
- SW1: footprint Button_Switch_THT:SW_DIP_SPSTx01_Slide_6.7x4.1mm_W7.62mm_P2.54mm_LowProfile -> Library:Slide Switch 3-pin
Changed lines of the file:
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@@
       (effects (font (size 1.524 1.524)))
     )
-    (property "Footprint" "Button_Switch_THT:SW_DIP_SPSTx01_Slide_6.7x4.1mm_W7.62mm_P2.54mm_LowProfile" (id 2) (at 246.38 54.61 0)
+    (property "Footprint" "Library:Slide Switch 3-pin" (id 2) (at 246.38 54.61 0)
       (effects (font (size 1.524 1.524)) hide)
     )
@@
     )
     (path "/e6c32bfe-2a10-452d-8622-3b0fb981ddf9"
-      (reference "SW1") (unit 1) (value "SWITCH") (footprint "Button_Switch_THT:SW_DIP_SPSTx01_Slide_6.7x4.1mm_W7.62mm_P2.54mm_LowProfile")
+      (reference "SW1") (unit 1) (value "SWITCH") (footprint "Library:Slide Switch 3-pin")
     )
     (path "/81316103-1aa7-4cdf-838f-26fdbe06c5b0"
