File: SidecarXE85/SidecarXE85-keyboard.kicad_pcb (KiCad board)
At the start: 2 copper layers, 164.3 x 133.4 mm, 63 parts, among them J2 Conn_02x08_Odd_Even, J3 Conn_01x04, SW1 Minus, SW10 1, SW11 Yes, SW12 F2, SW13 F4, SW14 LEFT, SW15 9, SW16 8, SW17 7, SW18 No, SW19 UP, SW2 Enter, SW20 DOWN, SW21 6, SW22 5, SW23 4, SW24 Del, SW25 RIGHT, SW26 Slash, SW27 Star, SW28 Plus, SW29 Esc, SW3 Period, SW30 TRIGGER, SW4 0, SW5 F1, SW6 F3, SW7 TRIGGER, SW8 3, SW9 2

Commit message: Sidecar keyboard board complete
Parts:
- added G***: LOGO, Library:ScreamingAtTheRadio, F.Cu at (41.0, 150.0)
- added G***: LOGO, LOGO, F.Cu at (135.2, 54.6)
- added REF**: KiCad-Logo2_5mm_SilkScreen, Symbol:KiCad-Logo2_5mm_SilkScreen, F.Cu at (65.0, 153.0)
- added REF**: OSHW-Logo2_7.3x6mm_SilkScreen, Symbol:OSHW-Logo2_7.3x6mm_SilkScreen, F.Cu at (82.0, 153.0)
Other:
- board text added: "Rev. 1 (c) Bertrand Le Roy 2023 https://github.com/bleroy/3d-junkyard/tree/main/SidecarXE85 https://atariage.com/forums/profile/76850-screamingattheradio/ https://www.youtube.com/@screamingattheradio"

Commit message: Sidecar XE85 prototype finalized
Changed lines of the file:
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@@
       (plotinvisibletext false)
       (sketchpadsonfab false)
-      (subtractmaskfromsilk false)
+      (subtractmaskfromsilk true)
       (outputformat 1)
       (mirror false)
-      (drillshape 1)
+      (drillshape 0)
       (scaleselection 1)
-      (outputdirectory "")
+      (outputdirectory "Fabrication/")
     )
   )
@@
     (at 135.15 54.5875)
     (attr board_only exclude_from_pos_files exclude_from_bom)
-    (fp_text reference "G***" (at 0 0) (layer "F.SilkS")
+    (fp_text reference "G***" (at 0 0) (layer "F.SilkS") hide
         (effects (font (size 1.5 1.5) (thickness 0.3)))
     )
@@
     (fp_line (start 13.28 5.1) (end 13.28 -22.88)
       (stroke (width 0.1) (type solid)) (layer "B.Fab"))
-    (pad "1" thru_hole roundrect (at 0 0 90) (size 1.7 1.7) (drill 1) (layers "*.Cu" "*.Mask") (roundrect_rratio 0.147059)
+    (pad "1" thru_hole roundrect (at 0 0 90) (size 1.7 1.7) (drill 1) (layers "*.Cu" "*.Mask") (roundrect_rratio 0.1470588235)
       (net 1 "COL1") (pinfunction "Pin_1") (pintype "passive"))
     (pad "2" thru_hole circle (at 2.54 0 90) (size 1.7 1.7) (drill 1) (layers "*.Cu" "*.Mask")
@@
     (fp_line (start 10 6.7) (end 10 -1.5)
       (stroke (width 0.1) (type solid)) (layer "B.Fab"))
-    (pad "1" thru_hole roundrect (at 0 0 270) (size 1.7 1.95) (drill 0.95) (layers "*.Cu" "*.Mask") (roundrect_rratio 0.147059)
+    (pad "1" thru_hole roundrect (at 0 0 270) (size 1.7 1.95) (drill 0.95) (layers "*.Cu" "*.Mask") (roundrect_rratio 0.1470588235)
       (net 17 "Net-(J3-Pin_1)") (pinfunction "Pin_1") (pintype "passive"))
     (pad "2" thru_hole oval (at 2.5 0 270) (size 1.7 1.95) (drill 0.95) (layers "*.Cu" "*.Mask")
