File: SidecarXE85/SidecarXE85.kicad_pcb (KiCad board)
At the start: 2 copper layers, 164.3 x 69.2 mm, 15 parts, among them J1 DE9_Plug, J2 DE9_Plug, J3 DE9_Receptacle, J4 Conn_02x08_Odd_Even, J5 DE9_Receptacle, SW1 SW_SPDT, U1 MM74C923, U2 74AHC04

Commit message: Sidecar XE85 prototype finalized
Parts:
- moved J5 5.54 mm to (168.9, 61.0)
- moved J3 5.54 mm to (168.9, 29.0)
- moved G*** 5.12 mm to (135.9, 17.1)
- moved REF** 2.29 mm to (107.3, 73.7)
- moved REF** 1.90 mm to (90.8, 73.7)
Routing:
- net Net-(J4-Pin_16): track 178.4 -> 172.8 mm
- net Net-(J4-Pin_15): track 172.6 -> 167.0 mm
- net Net-(J4-Pin_14): track 184.4 -> 178.8 mm
- net Net-(J4-Pin_13): track 166.2 -> 160.6 mm
- net Net-(J4-Pin_12): track 180.7 -> 175.1 mm
- net Net-(J4-Pin_11): track 177.1 -> 171.5 mm
- net Net-(J1-Pad9): track 156.4 -> 150.8 mm
- net Net-(J1-Pad6): track 156.4 -> 150.8 mm
- net Net-(J4-Pin_10): track 157.2 -> 151.6 mm
- net Net-(SW1-B): track 198.9 -> 193.4 mm
- net Net-(J2-Pad9): track 156.4 -> 150.8 mm
- net Net-(J2-Pad6): track 226.9 -> 221.4 mm
- net Net-(J2-Pad5): track 268.5 -> 262.9 mm
- net Net-(J2-Pad4): track 209.6 -> 204.1 mm
- net Net-(J2-Pad3): track 249.0 -> 243.4 mm
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