File: DecentXL/DecentXL-keyboard/DecentXL-keyboard.kicad_pcb (KiCad board)
At the start: 2 copper layers, 360 x 112 mm, 216 parts, among them J1 Conn_02x12_Odd_Even, J2 Conn_01x26, J3 Conn_01x04, J4 Conn_01x10, J5 Conn_01x10, J6 Conn_01x10, J7 Conn_01x10, SW0 SW_Push_45deg, SW1 SW_Push_45deg, SW2 SW_Push_45deg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

Commit message: DecentXL PCB progress
Parts:
- added REF**: Mousebites, DecentXL:Mousebites, F.Cu at (337.1, 105.9)
- added REF**: Mousebites, DecentXL:Mousebites, F.Cu at (337.1, 46.0)
- added REF**: Mousebites, DecentXL:Mousebites, F.Cu at (341.9, 105.9)
- added REF**: Mousebites, DecentXL:Mousebites, F.Cu at (341.9, 46.0)
- J2: footprint Connector_FFC-FPC:Molex_200528-0260_1x26-1MP_P1.00mm_Horizontal -> DecentXL:Molex_200528-0260_1x26-1MP_P1.00mm_Horizontal
- J3: footprint Connector_JST:JST_EH_S4B-EH_1x04_P2.50mm_Horizontal -> Connector_PinHeader_2.54mm:PinHeader_1x04_P2.54mm_Vertical; moved to B.Cu
- JP1: footprint Connector_PinHeader_2.54mm:PinHeader_1x02_P2.54mm_Vertical -> DecentXL:Potentiometer_CUI-PTN06-D02CB20
- JP2: footprint Connector_PinHeader_2.54mm:PinHeader_1x02_P2.54mm_Vertical -> Jumper:SolderJumper-2_P1.3mm_Bridged_RoundedPad1.0x1.5mm
- REF** (x3): footprint MountingHole:MountingHole_5.3mm_M5 -> DecentXL:MountingHole_5.3mm_M5
- SWCtlCaps1: footprint DecentXL:MX-2-00U-LED -> DecentXL:MX-2-00--1-75-U-LED
- SWEsc1: footprint DecentXL:MX-1-25U-LED -> DecentXL:MX-1-25--1-00-U-LED
- SWSpc1: footprint DecentXL:MX-6-25U-LED -> DecentXL:MX-9-00--6-25-U-LED
- SWTab1: footprint DecentXL:MX-1-75U-LED -> DecentXL:MX-1-75--1-50-U-LED
- moved J3 100.6 mm to (312.4, 26.9), turned to -90 degrees
- moved JP2 40.4 mm to (334.4, 97.7), turned to -90 degrees
- moved J1 26.8 mm to (328.4, 66.3), turned to 180 degrees
- moved JP1 14.4 mm to (315.4, 119.3), turned to -90 degrees
- moved R62 6.29 mm to (307.3, 28.9)
- moved SWFn2 3.57 mm to (82.5, 110.8)
- moved SWFn1 3.57 mm to (63.5, 110.8)
- moved SWCtl1 3.57 mm to (104.0, 110.8)
- moved J6 3.30 mm to (327.8, 26.7)
- moved J2 3.23 mm to (327.4, 89.2)
- moved J7 1.52 mm to (297.2, 22.9)
- moved REF** 1.19 mm to (330.6, 118.9)
- moved SWFn3 1.19 mm to (270.7, 110.8)
- moved SWFn4 1.19 mm to (289.7, 110.8)
- moved SWEsc1 1.19 mm to (44.4, 34.4)
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Other:
- board size 360 x 112 mm -> 357.6 x 112 mm
