File: DecentXL/DecentXL-keyboard/DecentXL-keyboard-modern.kicad_sch (KiCad schematic)
At the start: 199 parts, among them J1 Conn_02x12_Odd_Even, J2 Conn_01x26, J3 Conn_01x04, SW0 0, SW1 1, SW2 2, SW3 3, SW4 4, SW5 5, SW6 6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

Commit message: Fixing a mistake in XL rev.4m production files
Parts:
- D1: JLCPCB Part # C81598 -> C2286

Commit message: DecentXL Rev 4 vintage WIP
Parts:
- D1: footprint LED_SMD:LED_0201_0603Metric -> LED_SMD:LED_0603_1608Metric
Changed lines of the file:
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@@
       (effects (font (size 1.27 1.27)) (justify left))
     )
-    (property "Footprint" "LED_SMD:LED_0201_0603Metric" (at 198.12 154.94 0)
+    (property "Footprint" "LED_SMD:LED_0603_1608Metric" (at 198.12 154.94 0)
       (effects (font (size 1.27 1.27)) hide)
     )
