File: DecentXL/DecentXL-keyboard/DecentXL-keyboard-vintage.kicad_sch (KiCad schematic)
At the start: 211 parts, among them J1 Conn_02x12_Odd_Even, J2 Conn_01x26, J3 Conn_01x04, J4 Conn_01x10, J5 Conn_01x10, J6 Conn_01x10, SW0 0, SW1 1, SW2 2, SW3 3, SW4 4, SW5 5, SW6 6, SW6 7, SW8 8, SW9 9

Commit message: DecentXL Rev 4 vintage WIP
Parts:
- removed D1: LED, LED_SMD:LED_0201_0603Metric, symbol Device:LED
- removed D100, D101, D102, D103, D104, D105, D106, D107, D108, D109, D110, D111, D112, D113, D114, D115, D116, D117, D118, D119, D120, D121, D122, D123, D124, D125, D126, D127, D128, D69 (x2), D70, D71, D72, D73, D74, D75, D76, D77, D78, D79, D80, D81, D82, D83, D84, D85, D86, D87, D88, D89, D90, D91, D92, D93, D94, D95, D96, D97, D98, D99: 1N4148W, DecentXL:D_SOD-123, symbol Diode:1N4148W
- removed J4: Conn_01x10, Connector_PinHeader_2.54mm:PinHeader_1x10_P2.54mm_Vertical, symbol Connector_Generic:Conn_01x10
- removed J5, J6: Conn_01x10, Connector_FFC-FPC:Hirose_FH12-10S-0.5SH_1x10-1MP_P0.50mm_Horizontal, symbol Connector_Generic:Conn_01x10
- removed JP1, JP2: Jumper_3_Bridged12, Connector_PinHeader_2.54mm:PinHeader_1x03_P2.54mm_Horizontal, symbol Jumper:Jumper_3_Bridged12
- removed JP4: SolderJumper_2_Bridged, Jumper:SolderJumper-2_P1.3mm_Bridged_Pad1.0x1.5mm, symbol Jumper:SolderJumper_2_Bridged
- removed R2 (x2), R61 (x2), R62 (x2), R67: 100, DecentXL:R_0603_1608Metric, symbol Device:R
- removed SW6: 6, DecentXL:MX-1-00U-LED, symbol UniversalSwitchWithLED:SW_WITHLED
- removed SW6: 7, DecentXL:MX-1-00U-LED, symbol UniversalSwitchWithLED:SW_WITHLED
- removed SWBrk2: Break, DecentXL:MX-1-25U-LED, symbol UniversalSwitchWithLED:SW_WITHLED
- removed SWCtlCaps1: Caps, DecentXL:MX-2-00U-LED, symbol UniversalSwitchWithLED:SW_WITHLED
- removed SWDel2: Del, DecentXL:MX-2-00U-LED, symbol UniversalSwitchWithLED:SWITCH
- removed SWRet2: Return, DecentXL:MX-ISO-RETURN, symbol UniversalSwitchWithLED:SWITCH
- added D1, D10, D11, D12, D13, D14, D15, D16, D17, D18, D19, D20, D21, D22, D23, D24, D25, D26, D27, D28, D29, D3, D30, D31, D32, D33, D34, D35, D36, D37, D38, D39, D4, D40, D41, D42, D43, D44, D45, D46, D48, D49, D5, D50, D51, D52, D53, D54, D55, D56, D57, D58, D59, D6, D60, D61, D62, D7, D8, D9: 1N4148W, DecentXL:D_SOD-123, symbol Diode:1N4148W
- added D47: LED, LED_SMD:LED_0603_1608Metric, symbol Device:LED
- added JP1: SolderJumper_2_Bridged, Jumper:SolderJumper-2_P1.3mm_Bridged_Pad1.0x1.5mm, symbol Jumper:SolderJumper_2_Bridged
- added R1, R2, R60, R61, R62: 100, DecentXL:R_0603_1608Metric, symbol Device:R
- added SW6: 6, DecentXL:Choc-1-00U-LED, symbol UniversalSwitchWithLED:SW_WITHLED
- added SW7: 7, DecentXL:Choc-1-00U-LED, symbol UniversalSwitchWithLED:SW_WITHLED
- RV1: JLCPCB Rotation Offset 180 -> 270
- SW0, SW1, SW2, SW3, SW4, SW5, SW8, SW9, SWA1, SWB1, SWBrk1, SWC1, SWComma1, SWD1, SWDash1, SWDel1, SWE1, SWEqual1, SWF1, SWFn1, SWFn4, SWG1, SWGT1, SWH1, SWHlp1, SWI1, SWInv1, SWJ1, SWK1, SWL1, SWLT1, SWM1, SWN1, SWO1, SWOption1, SWP1, SWPeriod1, SWPlus1, SWQ1, SWR1, SWReset1, SWS1, SWSelect1, SWSemi1, SWSlash1, SWStar1, SWStart1, SWT1, SWU1, SWV1, SWW1, SWX1, SWY1, SWZ1: footprint DecentXL:MX-1-00U-LED -> DecentXL:Choc-1-00U-LED
- SWCps1, SWEsc1: footprint DecentXL:MX-1-25U-LED -> DecentXL:Choc-1-25U-LED
- SWCtl1: footprint DecentXL:MX-1-25U-LED -> DecentXL:Choc-1-75U-LED
- SWFn2: value F2 -> F3; footprint DecentXL:MX-1-00U-LED -> DecentXL:Choc-1-00U-LED
- SWFn3: value F3 -> F2; footprint DecentXL:MX-1-00U-LED -> DecentXL:Choc-1-00U-LED
- SWLeftSft1: footprint DecentXL:MX-2-25U-LED -> DecentXL:Choc-2-50U-LED
- SWRet1: footprint DecentXL:MX-1-50U-LED -> DecentXL:Choc-1-50U-LED; JLCPCB Rotation Offset 180 -> 270
- SWRightSft1: footprint DecentXL:MX-1-75U-LED -> DecentXL:Choc-1-75U-LED
- SWSpc1: footprint DecentXL:MX-6-25U-LED -> DecentXL:Choc-9-00U-LED
- SWTab1: footprint DecentXL:MX-1-75U-LED -> DecentXL:Choc-1-50U-LED
Connections:
- net CSL_GND is gone; now on net GND: SWOption1.2, SWReset1.2, SWSelect1.2, SWStart1.2
- net CSL_HELP is gone; now on net COL_2: SWHlp1.1
- net CSL_LED_GND is gone; now on net LED_GND: R11.2, R63.2, R64.2, R65.2, R66.2
- net CSL_OPTION is gone; now on net OPTION: SWOption1.1
- net CSL_RESET is gone; now on net RESET: SWReset1.1
- net CSL_SELECT is gone; now on net SELECT: SWSelect1.1
- net CSL_START is gone; now on net START: SWStart1.1
- net CSL_VCC_LED is gone; now on net VCC_LED: SWHlp1.4, SWOption1.4, SWReset1.4, SWSelect1.4, SWStart1.4
- net COL_1: now also SWFn2.1, SW6.1, SW7.1; no longer SWFn3.1
- net COL_8: now also SWFn3.1; no longer SWFn2.1
- net GND: now also D47.1 (K), JP1.1 (A)
- net LED_GND: now also JP1.2 (B), R1.2, R2.2, R60.2, R61.2, R62.2
- net PWR_LED: now also D47.2 (A)
- net ROW_1: now also D1.1 (K), D15.1 (K), D23.1 (K), D31.1 (K), D39.1 (K), D48.1 (K), D5.1 (K), D56.1 (K)
- net ROW_2: now also D16.1 (K), D24.1 (K), D32.1 (K), D40.1 (K), D49.1 (K), D57.1 (K), D6.1 (K)
- net ROW_3: now also D17.1 (K), D25.1 (K), D33.1 (K), D41.1 (K), D50.1 (K), D58.1 (K), D7.1 (K)
- net ROW_4: now also D18.1 (K), D26.1 (K), D34.1 (K), D42.1 (K), D51.1 (K), D59.1 (K), D8.1 (K)
- net ROW_5: now also D2.1 (K), D12.1 (K), D19.1 (K), D27.1 (K), D35.1 (K), D43.1 (K), D52.1 (K), D60.1 (K), D9.1 (K)
- net ROW_6: now also D13.1 (K), D20.1 (K), D28.1 (K), D36.1 (K), D44.1 (K), D53.1 (K), D61.1 (K)
- net ROW_7: now also D10.1 (K), D14.1 (K), D21.1 (K), D29.1 (K), D37.1 (K), D45.1 (K), D54.1 (K)
- net ROW_8: now also D11.1 (K), D22.1 (K), D3.1 (K), D30.1 (K), D38.1 (K), D4.1 (K), D46.1 (K), D55.1 (K), D62.1 (K)
- net VCC_LED: now also SW6.4, SW7.4
- net at SWK1.2: now also D19.2 (A)
- net at SWStar1.3: now also R56.1; no longer R48.1
- net at R49.1: now also SWS1.3; no longer SWA1.3
- net at SWDash1.2: now also D41.2 (A)
- net at SW0.2: now also D31.2 (A)
- net at R30.1: now also SWR1.3; no longer SWP1.3
- net at SWFn2.2: now also D11.2 (A)
- net at SWFn2.3: now also R12.1; no longer R56.1
- net at SWCtl1.2: now also D2.2 (A)
- net at SWF1.2: now also D28.2 (A)
- net at SWF1.3: now also R32.1; no longer R25.1
- net at R43.1: now also SWC1.3; no longer SWX1.3
- net at SWSemi1.2: now also D35.2 (A)
- net at SWLeftSft1.2, SWRightSft1.2: now also D3.2 (A)
- net at SWRightSft1.3: now also R4.1
- net at SWLT1.2: now also D39.2 (A)
- net at SWY1.3: now also R9.1; no longer R4.1
- net at SWO1.2: now also D25.2 (A)
- net at SW3.2: now also D32.2 (A)
- net at SW3.3: now also R37.1; no longer R29.1
- net at SWB1.2: now also D22.2 (A)
- net at R19.1: now also SW5.3; no longer SWB1.3
- net at SWHlp1.3: now also R5.1; no longer R11.1
- net at SW9.2: now also D23.2 (A)
- net at R20.1: now also SWI1.3; no longer SW9.3
- net at SWH1.2: now also D13.2 (A)
- net at R36.1: now also SW0.3; no longer SWLT1.3
- net at R14.1: now also SWJ1.3; no longer SWI1.3
- net at SWTab1.2: now also D59.2 (A)
- net at SWTab1.3: now also R63.1; no longer R55.1
- net at SWL1.3: now also R31.1; no longer R24.1
- net at SWFn3.3: now also R64.1; no longer R7.1
- net at R35.1: now also SWReset1.3; no longer SWC1.3
- net at SWT1.2: now also D18.2 (A)
- net at SWComma1.2: now also D29.2 (A)
- net at SWComma1.3: now also R33.1; no longer R26.1
- net at SWRet1.2: now also D58.2 (A)
- net at SWRet1.3: now also R62.1; no longer R54.1
- net at SWEqual1.2: now also D50.2 (A)
- net at SWA1.2: now also D53.2 (A)
- net at SWInv1.2: now also D54.2 (A)
- net at R50.1: now also SWSlash1.3; no longer SWInv1.3
- net at SWLeftSft1.3: now also R3.1
- net at SWPeriod1.2: now also D37.2 (A)
- net at SWN1.2: now also D10.2 (A)
- net at SWGT1.2: now also D48.2 (A)
- net at R44.1: now also SWLT1.3; no longer SWGT1.3
- net at SWSelect1.3: now also R17.1; no longer R64.1
- net at SWDash1.3: now also R46.1; no longer R38.1
- net at SWFn3.2: now also D60.2 (A)
- net at SWN1.3: now also R11.1; no longer R6.1
- net at SWEqual1.3: now also R54.1; no longer R46.1
- net at R28.1: now also SW4.3; no longer SW0.3
- net at SWPlus1.2: now also D43.2 (A)
- net at SWS1.2: now also D44.2 (A)
- net at R41.1: now also SWD1.3; no longer SWS1.3
- net at SWW1.2: now also D42.2 (A)
- net at SW5.2: now also D16.2 (A)
- net at SWD1.2: now also D36.2 (A)
- net at R65.1: now also SWCps1.3; no longer SWOption1.3
- net at SW1.2: now also D49.2 (A)
- net at R45.1: now also SW2.3; no longer SW1.3
- net at SWSpc1.3: now also R16.1; no longer R10.1
- net at SWG1.3: now also R23.1; no longer R17.1
- net at SWY1.2: now also D8.2 (A)
- net at SWSlash1.2: now also D45.2 (A)
- net at R8.1: now also SWU1.3; no longer SWJ1.3
- net at SWSemi1.3: now also R40.1; no longer R32.1
- net at SWPlus1.3: now also R48.1; no longer R40.1
- net at SWX1.2: now also D46.2 (A)
- net at SWG1.2: now also D20.2 (A)
- net at SWK1.3: now also R22.1; no longer R16.1
- net at SWStart1.3: now also R13.1; no longer R63.1
- net at SW2.2: now also D40.2 (A)
- net at SWL1.2: now also D27.2 (A)
- net at R42.1: now also SWPeriod1.3; no longer SWSlash1.3
- net at SWFn4.2: now also D62.2 (A)
- net at SWFn4.3: now also R66.1; no longer R58.1
- net at SW4.2: now also D24.2 (A)
- net at SWO1.3: now also R29.1; no longer R22.1
- net at SWDel1.2: now also D56.2 (A)
- net at R52.1: now also SWGT1.3; no longer SWDel1.3
- net at SW8.3: now also R18.1; no longer R12.1
- net at SWFn1.2: now also D9.2 (A)
- net at SWFn1.3: now also R10.1; no longer R5.1
- net at SWW1.3: now also R47.1; no longer R39.1
- net at R34.1: now also SWV1.3; no longer SWPeriod1.3
- net at R59.1: now also SWZ1.3; no longer SWCtl1.3
- net at SWQ1.2: now also D51.2 (A)
- net at SWQ1.3: now also R55.1; no longer R47.1
- net at SW8.2: now also D15.2 (A)
- net at SWEsc1.3: now also R61.1; no longer R53.1
- net at SWZ1.2: now also D55.2 (A)
- net at R51.1: now also SWX1.3; no longer SWZ1.3
- net at SWM1.2: now also D21.2 (A)
- net at SWM1.3: now also R24.1; no longer R18.1
- net at SWBrk1.2: now also D1.2 (A)
- net at SWE1.3: now also R39.1; no longer R31.1
- net at SWStar1.2: now also D52.2 (A)
- net at SWJ1.2: now also D12.2 (A)
- net at SWU1.2: now also D7.2 (A)
- net at SWP1.2: now also D33.2 (A)
- net at SWBrk1.3: now also R1.1
- net at SWI1.2: now also D17.2 (A)
- net at SWT1.3: now also R21.1; no longer R15.1
- net at SWCps1.2: now also D61.2 (A)
- net at SWC1.2: now also D38.2 (A)
- net at SWR1.2: now also D26.2 (A)
- net at SWV1.2: now also D30.2 (A)
- net at R27.1: now also SW9.3; no longer SWV1.3
- net at SWEsc1.2: now also D57.2 (A)
- net at R57.1: now also SWA1.3; no longer SWCps1.3
- net at SWE1.2: now also D34.2 (A)
- net at SWH1.3: now also R15.1; no longer R9.1
- net at SWHlp1.2: now also D4.2 (A)
- net at SWSpc1.2: now also D14.2 (A)
- new net: D6.2 (A), SW6.2
- new net: D5.2 (A), SW7.2
- new net: R2.1, SWCtl1.3
- new net: R25.1, SWB1.3
- new net: R58.1, SWInv1.3
- new net: R60.1, SWDel1.3
- new net: R53.1, SW1.3
- new net: R6.1, SW7.3
- new net: R7.1, SW6.3
- new net: R38.1, SWP1.3
- new net: R26.1, SWOption1.3
Other:
- title: DecentXL - Modern -> DecentXL - Vintage

Commit message: DecentXL Rev. 4 with separate vintage and modern versions
Parts:
- SWRet1: JLCPCB Rotation Offset 270 -> 180
Changed lines of the file:
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@@
       (effects (font (size 1.27 1.27)) hide)
     )
-    (property "JLCPCB Rotation Offset" "270" (at 218.44 46.99 0)
+    (property "JLCPCB Rotation Offset" "180" (at 218.44 46.99 0)
       (effects (font (size 1.27 1.27)) hide)
     )
