File: Decent400/Keyboard/Decent400.kicad_sch (KiCad schematic)
At the start: 181 parts, among them J1 Conn_01x02_Pin, J2 Conn_01x22, SW0 0, SW1 1, SW2 2, SW3 3, SW4 4, SW5 5, SW6 6, SW6 7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

Commit message: Finalizing Decent400 PCB
Parts:
- added R59: 100, Library:R_0603_1608Metric, symbol Device:R
- added SWCtl1: Control, Library:MX-1-25U-LED, symbol UniversalSwitchWithLED:SW_WITHLED
Connections:
- net COL_9: now also SWCtl1.1
- net GND: now also J2.22 (Pin_22); no longer J2.18 (Pin_18)
- net LED_GND: now also R59.2
- net OPTION: now also J2.19 (Pin_19); no longer J2.21 (Pin_21)
- net RESET: now also J2.18 (Pin_18); no longer J2.22 (Pin_22)
- net START: now also J2.21 (Pin_21); no longer J2.19 (Pin_19)
- net VCC_LED: now also SWCtl1.4
- net at D127.2 (A), SWCtl1.2: now also SWCtl1.2
- new net: R59.1, SWCtl1.3
- no-connect marks 2 -> 1
Changed lines of the file:
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@@
   (junction (at 186.69 67.31) (diameter 0) (color 0 0 0 0)
   )
+  (junction (at 64.77 66.04) (diameter 0) (color 0 0 0 0)
+  )
   (junction (at 217.17 34.29) (diameter 0) (color 0 0 0 0)
   )
@@
   (junction (at 240.03 39.37) (diameter 0) (color 0 0 0 0)
   )
+  (junction (at 74.93 85.09) (diameter 0) (color 0 0 0 0)
+  )
   (junction (at 227.33 29.21) (diameter 0) (color 0 0 0 0)
   )
@@
   (junction (at 217.17 62.23) (diameter 0) (color 0 0 0 0)
   )
+  (junction (at 81.28 81.28) (diameter 0) (color 0 0 0 0)
+  )
   (junction (at 189.23 99.06) (diameter 0) (color 0 0 0 0)
   )
@@
   (junction (at 139.7 72.39) (diameter 0) (color 0 0 0 0)
   )
+  (junction (at 74.93 76.2) (diameter 0) (color 0 0 0 0)
+  )
   (junction (at 158.75 114.3) (diameter 0) (color 0 0 0 0)
   )
@@
   (junction (at 167.64 123.19) (diameter 0) (color 0 0 0 0)
   )
-  (no_connect (at 138.43 179.07))
   (no_connect (at 34.29 148.59))
   (wire (pts (xy 240.03 123.19) (xy 240.03 129.54))
@@
     (stroke (width 0) (type default))
   )
-  (wire (pts (xy 64.77 20.32) (xy 64.77 76.2))
+  (wire (pts (xy 64.77 20.32) (xy 64.77 66.04))
     (stroke (width 0) (type default))
   )
@@
     (stroke (width 0) (type default))
   )
+  (wire (pts (xy 66.04 88.9) (xy 67.31 88.9))
+    (stroke (width 0) (type default))
+  )
   (wire (pts (xy 139.7 16.51) (xy 158.75 16.51))
     (stroke (width 0) (type default))
@@
     (stroke (width 0) (type default))
   )
+  (wire (pts (xy 81.28 81.28) (xy 110.49 81.28))
+    (stroke (width 0) (type default))
+  )
   (wire (pts (xy 234.95 86.36) (xy 234.95 90.17))
     (stroke (width 0) (type default))
@@
     (stroke (width 0) (type default))
   )
+  (wire (pts (xy 72.39 68.58) (xy 81.28 68.58))
+    (stroke (width 0) (type default))
+  )
   (wire (pts (xy 212.09 161.29) (xy 212.09 160.02))
     (stroke (width 0) (type default))
@@
     (stroke (width 0) (type default))
   )
+  (wire (pts (xy 74.93 85.09) (xy 74.93 88.9))
+    (stroke (width 0) (type default))
+  )
   (wire (pts (xy 162.56 78.74) (xy 162.56 83.82))
     (stroke (width 0) (type default))
@@
     (stroke (width 0) (type default))
   )
+  (wire (pts (xy 67.31 68.58) (xy 66.04 68.58))
+    (stroke (width 0) (type default))
+  )
   (wire (pts (xy 167.64 25.4) (xy 148.59 25.4))
     (stroke (width 0) (type default))
@@
     (stroke (width 0) (type default))
   )
+  (wire (pts (xy 64.77 66.04) (xy 64.77 76.2))
+    (stroke (width 0) (type default))
+  )
   (wire (pts (xy 237.49 29.21) (xy 237.49 43.18))
     (stroke (width 0) (type default))
@@
     (stroke (width 0) (type default))
   )
+  (wire (pts (xy 66.04 68.58) (xy 66.04 88.9))
+    (stroke (width 0) (type default))
+  )
   (wire (pts (xy 205.74 39.37) (xy 224.79 39.37))
     (stroke (width 0) (type default))
@@
     (stroke (width 0) (type default))
   )
+  (wire (pts (xy 74.93 66.04) (xy 74.93 76.2))
+    (stroke (width 0) (type default))
+  )
   (wire (pts (xy 245.11 160.02) (xy 245.11 161.29))
     (stroke (width 0) (type default))
@@
     (stroke (width 0) (type default))
   )
+  (wire (pts (xy 81.28 68.58) (xy 81.28 81.28))
+    (stroke (width 0) (type default))
+  )
   (wire (pts (xy 86.36 64.77) (xy 86.36 69.85))
     (stroke (width 0) (type default))
@@
     (stroke (width 0) (type default))
   )
-  (wire (pts (xy 72.39 81.28) (xy 110.49 81.28))
+  (wire (pts (xy 72.39 81.28) (xy 81.28 81.28))
     (stroke (width 0) (type default))
   )
@@
     )
   )
-  (global_label "OPTION" (shape output) (at 128.27 152.4 270) (fields_autoplaced)
+  (global_label "OPTION" (shape output) (at 123.19 152.4 270) (fields_autoplaced)
     (effects (font (size 1.27 1.27)) (justify right))
-    (property "Intersheetrefs" "${INTERSHEET_REFS}" (at 128.27 162.2191 90)
+    (property "Intersheetrefs" "${INTERSHEET_REFS}" (at 123.19 162.2191 90)
       (effects (font (size 1.27 1.27)) (justify right) hide)
     )
@@
     )
   )
-  (global_label "RESET" (shape output) (at 130.81 152.4 270) (fields_autoplaced)
+  (global_label "RESET" (shape output) (at 120.65 152.4 270) (fields_autoplaced)
     (effects (font (size 1.27 1.27)) (justify right))
-    (property "Intersheetrefs" "${INTERSHEET_REFS}" (at 130.81 161.1303 90)
+    (property "Intersheetrefs" "${INTERSHEET_REFS}" (at 120.65 161.1303 90)
       (effects (font (size 1.27 1.27)) (justify right) hide)
     )
@@
     )
   )
-  (global_label "START" (shape output) (at 123.19 152.4 270) (fields_autoplaced)
+  (global_label "START" (shape output) (at 128.27 152.4 270) (fields_autoplaced)
     (effects (font (size 1.27 1.27)) (justify right))
-    (property "Intersheetrefs" "${INTERSHEET_REFS}" (at 123.19 160.8885 90)
+    (property "Intersheetrefs" "${INTERSHEET_REFS}" (at 128.27 160.8885 90)
       (effects (font (size 1.27 1.27)) (justify right) hide)
     )
@@
     )
   )
-  (global_label "GND" (shape input) (at 120.65 152.4 270) (fields_autoplaced)
+  (global_label "GND" (shape input) (at 130.81 152.4 270) (fields_autoplaced)
     (effects (font (size 1.27 1.27)) (justify right))
-    (property "Intersheetrefs" "${INTERSHEET_REFS}" (at 120.65 159.2557 90)
+    (property "Intersheetrefs" "${INTERSHEET_REFS}" (at 130.81 159.2557 90)
       (effects (font (size 1.27 1.27)) (justify right) hide)
     )
@@
     )
   )
+  (symbol (lib_id "Device:R") (at 71.12 88.9 90) (unit 1)
+    (in_bom yes) (on_board yes) (dnp no)
+    (property "Reference" "R59" (at 71.12 88.9 90)
+      (effects (font (size 1.27 1.27)))
+    )
+    (property "Value" "100" (at 71.12 86.7211 90)
+      (effects (font (size 1.27 1.27)) hide)
+    )
+    (property "Footprint" "Library:R_0603_1608Metric" (at 71.12 90.678 90)
+      (effects (font (size 1.27 1.27)) hide)
+    )
+    (property "Datasheet" "~" (at 71.12 88.9 0)
+      (effects (font (size 1.27 1.27)) hide)
+    )
+    (property "JLCPCB Part #" "C22775" (at 71.12 88.9 0)
+      (effects (font (size 1.27 1.27)) hide)
+    )
+    (property "JLCPCB Rotation Offset" "" (at 71.12 88.9 0)
+      (effects (font (size 1.27 1.27)) hide)
+    )
+    (pin "1")
+    (pin "2")
+    (instances
+      (project "DecentXE"
+        (path "/2f215f15-3d52-4c91-93e6-3ea03a95622f"
+          (reference "R59") (unit 1)
+        )
+      )
+      (project "Decent800"
+        (path "/89eaabff-fda3-406f-879a-3ecedd6e1b7a"
+          (reference "R3") (unit 1)
+        )
+      )
+      (project "DecentXL-keyboard"
+        (path "/a9892182-6906-43e4-9038-45744b4ac951"
+          (reference "R60") (unit 1)
+        )
+      )
+      (project "Decent400"
+        (path "/bb8bfa28-ab9e-4457-bbf1-e505aca6ff00"
+          (reference "R3") (unit 1)
+        )
+      )
+    )
+  )
   (symbol (lib_name "1N4148W_48") (lib_id "Diode:1N4148W") (at 173.99 76.2 180) (unit 1)
     (in_bom yes) (on_board yes) (dnp no) (fields_autoplaced)
@@
   (symbol (lib_id "UniversalSwitchWithLED:SW_WITHLED") (at 222.25 20.32 0) (unit 1)
     (in_bom yes) (on_board yes) (dnp no)
-    (property "Reference" "SWDel1" (at 227.33 21.59 0)
+    (property "Reference" "SWDel1" (at 220.98 17.78 0)
       (effects (font (size 1 1)))
     )
@@
         )
       )
+    )
+  )
+  (symbol (lib_id "UniversalSwitchWithLED:SW_WITHLED") (at 69.85 66.04 0) (unit 1)
+    (in_bom yes) (on_board yes) (dnp no)
+    (property "Reference" "SWCtl1" (at 69.85 63.5 0)
+      (effects (font (size 1.27 1.27)))
+    )
+    (property "Value" "Control" (at 69.85 61.214 0)
+      (effects (font (size 1.27 1.27)) hide)
+    )
+    (property "Footprint" "Library:MX-1-25U-LED" (at 69.85 66.04 0)
+      (effects (font (size 1.524 1.524)) hide)
+    )
+    (property "Datasheet" "~" (at 69.85 66.04 0)
+      (effects (font (size 1.524 1.524)) hide)
+    )
+    (property "JLCPCB Part #" "C193191" (at 69.85 66.04 0)
+      (effects (font (size 1.27 1.27)) hide)
+    )
+    (property "JLCPCB Rotation Offset" "180" (at 69.85 66.04 0)
+      (effects (font (size 1.27 1.27)) hide)
+    )
+    (pin "1")
+    (pin "2")
+    (pin "3")
+    (pin "4")
+    (instances
+      (project "DecentXE"
+        (path "/2f215f15-3d52-4c91-93e6-3ea03a95622f"
+          (reference "SWCtl1") (unit 1)
+        )
+      )
+      (project "Decent800"
+        (path "/89eaabff-fda3-406f-879a-3ecedd6e1b7a"
+          (reference "SWCtl1") (unit 1)
+        )
+      )
+      (project "DecentXL-keyboard"
+        (path "/a9892182-6906-43e4-9038-45744b4ac951"
+          (reference "SWCtl1") (unit 1)
+        )
+      )
+      (project "Decent400"
+        (path "/bb8bfa28-ab9e-4457-bbf1-e505aca6ff00"
+          (reference "SWCtl2") (unit 1)
+        )
+      )

Commit message: Decent400 & 800 production files, dir cleanups
Parts:
- SWRet1: JLCPCB Rotation Offset 180 -> 90
Changed lines of the file:
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@@
       (effects (font (size 1.27 1.27)) hide)
     )
-    (property "JLCPCB Rotation Offset" "180" (at 222.25 48.26 0)
+    (property "JLCPCB Rotation Offset" "90" (at 222.25 48.26 0)
       (effects (font (size 1.27 1.27)) hide)
     )
