File: Decent400/Keyboard/Decent400-Wide.kicad_sch (KiCad schematic)
At the start: 182 parts, among them J1 Conn_01x02_Pin, J2 Conn_01x22, SW0 0, SW1 1, SW2 2, SW3 3, SW4 4, SW5 5, SW6 6, SW6 7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

Commit message: Decent400 Wide + enclosure + USB adapter
Parts:
- added R3: 100, Library:R_0603_1608Metric, symbol Device:R
Connections:
- net GND: now also R3.2; no longer D57.1 (K)
- new net: D57.1 (K), R3.1
