File: Decent1200/Plate/Decent1200-plate.kicad_pcb (KiCad board)
At the start: 2 copper layers, 291.5 x 138.5 mm, 56 parts, among them SW0 0, SW1 1, SW2 2, SW3 3, SW4 4, SW5 5, SW6 6, SW7 7, SW8 8, SW9 9

Commit message: Decent1200 PCB and plate finalization
Parts:
- removed the G*** at (97.6, 134.2)
- removed the REF** at (286.8, 132.1)
- added G***: LOGO, LOGO, F.Cu at (101.1, 133.4)
- added G***: DECENT 1200, LOGO, F.Cu at (75.1, 49.9)
- added REF**: MountingHole_2.2mm_M2, MountingHole:MountingHole_2.2mm_M2, F.Cu at (337.5, 50.0)
- added REF**: KiCad-Logo2_5mm_SilkScreen, Symbol:KiCad-Logo2_5mm_SilkScreen, F.Cu at (285.8, 132.7)
- added REF**: MountingHole_2.2mm_M2, MountingHole:MountingHole_2.2mm_M2, F.Cu at (53.0, 50.0)
Other:
- board size 291.5 x 138.5 mm -> 291.5 x 102.4 mm
- board text added: "Decent 1200 Keyboard rev. 1 © Bertrand Le Roy 2023 https://github.com/bleroy/3d-junkyard/tree/main/Decent1200 https://atariage.com/forums/profile/76850-screamingattheradio/ https://www.youtube.com/@ScreamingAtTheRadio"
- board text removed: "Decent 1200 Keyboard rev. 1 © Bertrand Le Roy 2023 https://github.com/bleroy/3d-junkyard/tree/main/Decent1200 https://atariage.com/forums/profile/76850-screamingattheradio/ https://www.twitch.tv/screamingattheradio https://www.youtube.com/@ScreamingAtTheRadio"

Commit message: Decent1200 plate rev. 2
Parts:
- moved G*** 123.1 mm to (166.7, 132.2)
- moved REF** 107.5 mm to (178.9, 144.2)
- moved G*** 51.6 mm to (151.6, 144.3)
- moved REF** 35.5 mm to (302.4, 55.5)
- moved REF** 21.5 mm to (73.8, 55.5)
Other:
- board size 291.5 x 102.4 mm -> 290.5 x 95.3 mm
- board text added: "Decent 1200 Keyboard rev. 2 © Bertrand Le Roy 2023 www.youtube.com/@ScreamingAtTheRadio github.com/bleroy/3d-junkyard/tree/main/Decent1200 atariage.com/forums/profile/76850-screamingattheradio/"
- board text removed: "Decent 1200 Keyboard rev. 1 © Bertrand Le Roy 2023 https://github.com/bleroy/3d-junkyard/tree/main/Decent1200 https://atariage.com/forums/profile/76850-screamingattheradio/ https://www.youtube.com/@ScreamingAtTheRadio"

Commit message: Decent 1200 rev. 2 production files
Parts:
- moved G*** 56.4 mm to (223.1, 132.1)
- moved G*** 11.8 mm to (154.1, 132.8)
- moved REF** 11.6 mm to (178.8, 132.6)
Other:
- board text removed: "Space"

Commit message: Decent1200 Rev. 3
Other:
- board size 290.5 x 95.3 mm -> 288.1 x 95.3 mm
- board text added: "Decent 1200 Keyboard rev. 3 © Bertrand Le Roy 2023 www.youtube.com/@ScreamingAtTheRadio github.com/bleroy/3d-junkyard/tree/main/Decent1200 atariage.com/forums/profile/76850-screamingattheradio/"
- board text removed: "Decent 1200 Keyboard rev. 2 © Bertrand Le Roy 2023 www.youtube.com/@ScreamingAtTheRadio github.com/bleroy/3d-junkyard/tree/main/Decent1200 atariage.com/forums/profile/76850-screamingattheradio/"

Commit message: Decent1200 plate Rev. 3
Parts:
- removed SWCtlCaps1: ControlCaps, Library:MX-1-75--2-00U-Hole
- removed SWLeftSft1: Shift, Library:MX-2-25U--2-50-Hole
Other:
- outline, holes or cut-outs redrawn
