File: Decent800/Plate/Decent800-plate.kicad_pcb (KiCad board)
At the start: 2 copper layers, 285.9 x 95.4 mm, 66 parts, among them SW0 0, SW1 1, SW2 2, SW3 3, SW4 4, SW5 5, SW6 6, SW7 7, SW8 8, SW9 9

Commit message: Decent800 fixes
Parts:
- SWRet1: footprint Library:MX-1-50U-Hole -> Library:MX-1-50U-Hole-Right
Changed lines of the file:
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@@
     (at 44.69275 56.972)
     (descr "1.5U MX switch metal plate hole")
-    (tags "MX keyswitch 1.00u PCB")
+    (tags "MX keyswitch 1.50u PCB")
     (property "JLCPCB Part #" "C193191")
     (property "JLCPCB Rotation Offset" "180")
@@
         (effects (font (size 1.5 1.5) (thickness 0.3)))
     )
-    (fp_poly
-      (pts
-        (xy -20 2.5)
-        (xy -15 -2.5)
-        (xy 20.1 -2.5)
-        (xy 15.2 2.5)
-      )
-      (stroke (width 0.1) (type solid)) (fill solid) (layer "F.Cu"))
     (fp_poly
       (pts
@@
       )
       (stroke (width 0) (type solid)) (fill solid) (layer "F.Cu"))
+    (fp_poly
+      (pts
+        (xy -20 2.5)
+        (xy -15 -2.5)
+        (xy 20.1 -2.5)
+        (xy 15.2 2.5)
+      )
+      (stroke (width 0.1) (type solid)) (fill solid) (layer "F.Mask"))
   )
   (footprint "Library:MX-1-00U-Hole" (layer "F.Cu")
@@
     )
   )
-  (footprint "Library:MX-1-50U-Hole" (layer "F.Cu")
+  (footprint "Library:MX-1-50U-Hole-Right" (layer "F.Cu")
     (at 301.86775 56.972)
-    (descr "1.5U MX switch metal plate hole")
+    (descr "1.5U MX switch metal plate hole - right side version")
     (tags "MX keyswitch 1.50u PCB")
     (property "JLCPCB Part #" "C193191")
@@
     (property "Sheetname" "")
     (attr through_hole)
-    (fp_text reference "SWRet1" (at 0 -7.874) (layer "Cmts.User") hide
-        (effects (font (size 1 1) (thickness 0.15)))
-    )
-    (fp_text value "Return" (at 0 7.874) (layer "F.Fab") hide
+    (fp_text reference "SWRet1" (at 0 7.874 180) (layer "Cmts.User") hide
+        (effects (font (size 1 1) (thickness 0.15)))
+    )
+    (fp_text value "Return" (at 0 -7.874 180) (layer "F.Fab") hide
         (effects (font (size 1 1) (thickness 0.15)))
     )
@@
     (fp_line (start 14.2875 9.525) (end -14.2875 9.525)
       (stroke (width 0.15) (type solid)) (layer "F.SilkS"))
-    (fp_line (start -7 -7) (end -7 7)
-      (stroke (width 0.12) (type solid)) (layer "Edge.Cuts"))
-    (fp_line (start -7 -7) (end 11.7625 -7)
-      (stroke (width 0.12) (type solid)) (layer "Edge.Cuts"))
-    (fp_line (start -7 7) (end 11.7625 7)
-      (stroke (width 0.12) (type solid)) (layer "Edge.Cuts"))
-    (fp_line (start 11.7625 -7) (end 11.7625 7)
+    (fp_line (start -11.7625 7) (end -11.7625 -7)
+      (stroke (width 0.12) (type solid)) (layer "Edge.Cuts"))
+    (fp_line (start 7 -7) (end -11.7625 -7)
+      (stroke (width 0.12) (type solid)) (layer "Edge.Cuts"))
+    (fp_line (start 7 7) (end -11.7625 7)
+      (stroke (width 0.12) (type solid)) (layer "Edge.Cuts"))
+    (fp_line (start 7 7) (end 7 -7)
       (stroke (width 0.12) (type solid)) (layer "Edge.Cuts"))
     (model "${KISYS3DMOD}/Button_Switch_Keyboard.3dshapes/SW_Cherry_MX_1.00u_PCB.wrl"
@@
     (at 49.45525 76.022)
     (descr "1.5U MX switch metal plate hole")
-    (tags "MX keyswitch 1.00u PCB")
-    (property "JLCPCB Part #" "C193191")
-    (property "JLCPCB Rotation Offset" "180")
+    (tags "MX keyswitch 1.50u PCB")
+    (property "JLCPCB Part #" "C193191")
+    (property "JLCPCB Rotation Offset" "180")

Commit message: Finalize Decent800 PCB and plate
Parts:
- removed SWBrk1: Break, Library:MX-1-00U-Hole
- removed SWDel1: Del, Library:MX-1-00U-Hole
- added REF**: MX_Hole_2.00, Library:MX-2-00U-Hole, F.Cu at (297.1, 37.9)

Commit message: Decent800 rev. 2
Other:
- board text added: "Decent 800 rev. 2 © Bertrand Le Roy 2023 github.com/bleroy/3d-junkyard/tree/main/Decent800 atariage.com/forums/profile/76850-screamingattheradio/"
- board text removed: "Decent 800 rev. 1 © Bertrand Le Roy 2023 github.com/bleroy/3d-junkyard/tree/main/Decent800 atariage.com/forums/profile/76850-screamingattheradio/"
