File: Decent400/Plate/Decent400-plate-wide.kicad_pcb (KiCad board)
At the start: 2 copper layers, 314.3 x 97 mm, 69 parts, among them SW0 0, SW1 1, SW2 2, SW3 3, SW4 4, SW5 5, SW6 6, SW7 7, SW8 8, SW9 9

Commit message: Decent400 Wide + enclosure + USB adapter
Other:
- outline, holes or cut-outs redrawn
