File: Decent400/Plate/Decent400-plate-inner.kicad_pcb (KiCad board)
At the start: 2 copper layers, 252.6 x 93.5 mm, 62 parts, among them SW0 0, SW1 1, SW2 2, SW3 3, SW4 4, SW5 5, SW6 6, SW7 7, SW8 8, SW9 9

Commit message: Decent 400i routed
Other:
- outline, holes or cut-outs redrawn
- board text added: "Backlight"
- board text removed: "^"

Commit message: Decent400 internal ready for prod
Routing:
- added copper zone on B.Cu, net (none)
- added copper zone on F.Cu, net (none)
Changed lines of the file:
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@@
+		)
+	)
+	(zone
+		(net 0)
+		(net_name "")
+		(layers "F&B.Cu")
+		(hatch edge 0.5)
+		(connect_pads
+			(clearance 0.5)
+		)
+		(min_thickness 0.25)
+		(filled_areas_thickness no)
+		(fill yes
+			(thermal_gap 0.5)
+			(thermal_bridge_width 0.5)
+			(island_removal_mode 1)
+			(island_area_min 10)
+		)
+		(polygon
+			(pts
+				(xy 25.3925 31.552532) (xy 281.9325 31.552532) (xy 281.9325 128.072532) (xy 25.3925 128.072532)
+			)
 		)
 	)
