File: Decent400/Plate/Decent400-plate.kicad_pcb (KiCad board)
At the start: 2 copper layers, 252.6 x 93.5 mm, 60 parts, among them SW0 0, SW1 1, SW2 2, SW3 3, SW4 4, SW5 5, SW6 6, SW7 7, SW8 8, SW9 9

Commit message: Decent400 rev.5
The one with only one space bar...
Other:
- board text added: "Decent 400 rev. 5 © Bertrand Le Roy 2026"
- board text removed: "Decent 400 rev. 4.2i © Bertrand Le Roy 2026"
