File: DecentXL/DecentXL-plate/DecentXL-plate-modern.kicad_pcb (KiCad board)
At the start: 2 copper layers, 291.6 x 103.5 mm, 101 parts, among them SW0 SW_Push_45deg, SW1 SW_Push_45deg, SW2 SW_Push_45deg, SW3 SW_Push_45deg, SW4 SW_Push_45deg, SW5 SW_Push_45deg, SW6 SW_Push_45deg, SW7 SW_Push_45deg, SW8 SW_Push_45deg, SW9 SW_Push_45deg

Commit message: DecentXL Rev. 4 with separate vintage and modern versions
Parts:
- moved SWBrk1 2.38 mm to (248.8, 114.5)
- moved SWFn4 2.38 mm to (289.3, 114.5)
- moved SWCtl1 2.38 mm to (103.6, 114.5)
- moved SWFn1 2.38 mm to (63.1, 114.5)
- moved SWFn2 2.38 mm to (82.2, 114.5)
- moved SWSpc1 2.38 mm to (176.2, 114.5)
- moved SWFn3 2.38 mm to (270.3, 114.5)
- moved G*** 2.04 mm to (44.0, 111.5)

Commit message: Some version catch-up, and 800 readme
Other:
- board text added: "Rev. 4.1m (c) Bertrand Le Roy 2023 github.com/bleroy/3d-junkyard/DecentXL youtube.com/@screamingattheradio"
- board text removed: "Rev. 4m (c) Bertrand Le Roy 2023 github.com/bleroy/3d-junkyard/DecentXL youtube.com/@screamingattheradio"
