File: DecenTKL/Keyboard/key.kicad_sch (KiCad schematic)
At the start: 4 parts, among them SW17 SW_Push

Commit message: DecenTKL numpad update
Parts:
- C16: value 104 -> 100nF; JLCPCB Part # C83054 -> C14663
- D32: footprint DecenTKL:SK6812 MINI-EA -> LED_SMD:LED_SK6812MINI_PLCC4_3.5x3.5mm_P1.75mm; symbol LED:SK6812MINI -> DecentUSB_Library:SK6812MINI
Connections:
- net GND: now also D32.3 (VSS); no longer D32.2 (VSS)
- net RGB_IN: now also D32.4 (DIN); no longer D32.3 (DIN)
- net RGB_OUT: now also D32.2 (DOUT); no longer D32.1 (DOUT)
- net VBUS: now also D32.1 (VDD); no longer D32.4 (VDD)
Changed lines of the file:
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@@
+			)
+		)
+		(property "JLCPCB Position Offset" ""
+			(at 132.08 93.98 0)
+			(effects
+				(font
+					(size 1.27 1.27)
+				)
+				(hide yes)
 			)
 		)
@@
 				(path "/2c073ed7-8422-482e-9fe5-a73c0717c131/7628d00f-9e3d-4cab-b942-743bdaf9e232"
 					(reference "D35")
-					(unit 1)
-				)
-				(path "/2c073ed7-8422-482e-9fe5-a73c0717c131/80e70f0e-f533-4345-82eb-6ed67d3f0d54"
-					(reference "D1")
 					(unit 1)
 				)
@@
 		(dnp no)
 		(fields_autoplaced yes)
-		(property "Reference" "#PWR070"
+		(property "Reference" "#PWR068"
 			(at 179.07 109.22 0)
 			(effects
@@
 		(dnp no)
 		(fields_autoplaced yes)
-		(property "Reference" "#PWR077"
+		(property "Reference" "#PWR090"
 			(at 179.07 91.44 0)
 			(effects
@@
 			)
 		)
-		(property "Value" "104"
+		(property "Value" "100nF"
 			(at 181.991 96.4621 0)
 			(effects
@@
 			)
 		)
-		(property "JLCPCB Part #" " C83054"
+		(property "JLCPCB Part #" "C14663"
 			(at 179.07 95.25 0)
 			(effects
@@
 		)
 		(property "JLCPCB Rotation Offset" ""
+			(at 179.07 95.25 0)
+			(effects
+				(font
+					(size 1.27 1.27)
+				)
+				(hide yes)
+			)
+		)
+		(property "JLCPCB Position Offset" ""
 			(at 179.07 95.25 0)
 			(effects
@@
 				(path "/2c073ed7-8422-482e-9fe5-a73c0717c131/7628d00f-9e3d-4cab-b942-743bdaf9e232"
 					(reference "C18")
-					(unit 1)
-				)
-				(path "/2c073ed7-8422-482e-9fe5-a73c0717c131/80e70f0e-f533-4345-82eb-6ed67d3f0d54"
-					(reference "C1")
 					(unit 1)
 				)
@@
 			)
 		)
+		(property "JLCPCB Position Offset" ""
+			(at 127 97.79 0)
+			(effects
+				(font
+					(size 1.27 1.27)
+				)
+				(hide yes)
+			)
+		)
 		(pin "1"
 		)
@@
 					(unit 1)
 				)
-				(path "/2c073ed7-8422-482e-9fe5-a73c0717c131/80e70f0e-f533-4345-82eb-6ed67d3f0d54"
-					(reference "SW2")
-					(unit 1)
-				)
 				(path "/2c073ed7-8422-482e-9fe5-a73c0717c131/8ad9e23f-c013-482d-8b93-6b9c6e6b27e1"
 					(reference "SW12")
@@
 	)
 	(symbol
-		(lib_id "LED:SK6812MINI")
+		(lib_id "DecentUSB_Library:SK6812MINI")
 		(at 157.48 95.25 0)
 		(unit 1)
@@
 			)
 		)
-		(property "Footprint" "DecenTKL:SK6812 MINI-EA"
+		(property "Footprint" "LED_SMD:LED_SK6812MINI_PLCC4_3.5x3.5mm_P1.75mm"
 			(at 158.75 102.87 0)
 			(effects
@@
 			(at 157.48 95.25 0)
 			(effects
+				(font
+					(size 1.27 1.27)
+				)
+				(hide yes)
+			)
+		)
+		(property "JLCPCB Position Offset" ""
+			(at 157.48 95.25 0)
+			(effects

Commit message: DecenTKL NumPad WIP
Parts:
- SW17: value SW_Push -> MX; JLCPCB Layer Override (none) -> B.Cu; JLCPCB Part # C5333465 -> C5156480
Changed lines of the file:
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@@
+			)
+		)
+		(property "JLCPCB Layer Override" ""
+			(at 132.08 93.98 0)
+			(effects
+				(font
+					(size 1.27 1.27)
+				)
+				(hide yes)
 			)
 		)
@@
 			)
 		)
+		(property "JLCPCB Layer Override" ""
+			(at 179.07 95.25 0)
+			(effects
+				(font
+					(size 1.27 1.27)
+				)
+				(hide yes)
+			)
+		)
 		(pin "1"
 		)
@@
 			)
 		)
-		(property "Value" "SW_Push"
+		(property "Value" "MX"
 			(at 127 93.1488 0)
 			(effects
@@
 			)
 		)
-		(property "JLCPCB Part #" "C5333465"
+		(property "JLCPCB Part #" "C5156480"
 			(at 127 97.79 0)
 			(effects
@@
 		)
 		(property "JLCPCB Position Offset" ""
+			(at 127 97.79 0)
+			(effects
+				(font
+					(size 1.27 1.27)
+				)
+				(hide yes)
+			)
+		)
+		(property "JLCPCB Layer Override" "B.Cu"
 			(at 127 97.79 0)
 			(effects
@@
 			(at 157.48 95.25 0)
 			(effects
+				(font
+					(size 1.27 1.27)
+				)
+				(hide yes)
+			)
+		)
+		(property "JLCPCB Layer Override" ""
+			(at 157.48 95.25 0)
+			(effects
