File: DecenTKL/NumPad/2040.kicad_sch (KiCad schematic)
At the start: 25 parts, among them U1 NCP1117-3.3_SOT223, U2 W25Q128JVS, U3 RP2040, Y1 ABM8-272-T3

Commit message: DecenTKL numpad update
Parts:
- R1, R2: JLCPCB Part # C874875 -> C103492
- R3: now left out of the parts list
- U1: JLCPCB Rotation Offset (none) -> 180
- U2: JLCPCB Rotation Offset (none) -> 270
