File: DecenTKL/NumPad/RGB.kicad_sch (KiCad schematic)
At the start: 2 parts

Commit message: DecenTKL numpad update
Parts:
- C36: value 104 -> 100nF; JLCPCB Part # C83054 -> C14663
- D39: renamed from D40; footprint DecenTKL:SK6812 MINI-EA -> LED_SMD:LED_SK6812MINI_PLCC4_3.5x3.5mm_P1.75mm; symbol LED:SK6812MINI -> DecentUSB_Library:SK6812MINI
Connections:
- net GND: now also D39.3 (VSS); no longer D39.2 (VSS)
- net RGB_IN: now also D39.4 (DIN); no longer D39.3 (DIN)
- net RGB_OUT: now also D39.2 (DOUT); no longer D39.1 (DOUT)
- net VBUS: now also D39.1 (VDD); no longer D39.4 (VDD)
Changed lines of the file:
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@@
 			)
 		)
-		(property "Value" "104"
+		(property "Value" "100nF"
 			(at 161.671 90.1121 0)
 			(effects
@@
 			)
 		)
-		(property "JLCPCB Part #" " C83054"
+		(property "JLCPCB Part #" "C14663"
 			(at 158.75 88.9 0)
 			(effects
@@
 		)
 		(property "JLCPCB Rotation Offset" ""
+			(at 158.75 88.9 0)
+			(effects
+				(font
+					(size 1.27 1.27)
+				)
+				(hide yes)
+			)
+		)
+		(property "JLCPCB Position Offset" ""
 			(at 158.75 88.9 0)
 			(effects
@@
 	)
 	(symbol
-		(lib_id "LED:SK6812MINI")
+		(lib_id "DecentUSB_Library:SK6812MINI")
 		(at 137.16 88.9 0)
 		(unit 1)
@@
 		(dnp no)
 		(fields_autoplaced yes)
-		(property "Reference" "D40"
+		(property "Reference" "D39"
 			(at 148.7677 82.755 0)
 			(effects
@@
 			)
 		)
-		(property "Footprint" "DecenTKL:SK6812 MINI-EA"
+		(property "Footprint" "LED_SMD:LED_SK6812MINI_PLCC4_3.5x3.5mm_P1.75mm"
 			(at 138.43 96.52 0)
 			(effects
@@
 			(at 137.16 88.9 0)
 			(effects
+				(font
+					(size 1.27 1.27)
+				)
+				(hide yes)
+			)
+		)
+		(property "JLCPCB Position Offset" ""
+			(at 137.16 88.9 0)
+			(effects
