File: DecenTKL/NumPad/DecentNumPad.kicad_sch (KiCad schematic)
At the start: 4 parts, among them J1 Joystick1, J2 Joystick2, J3 Conn_02x20_Counter_Clockwise, SW1 BOOTSEL

Commit message: DecenTKL numpad update
Parts:
- J1, J2, J3, SW1: now left out of the parts list
Other:
- sheet Eight: file ../../Keyboard/key.kicad_sch -> ../Keyboard/key.kicad_sch
- sheet Enter: file ../../Keyboard/key.kicad_sch -> ../Keyboard/key.kicad_sch
- sheet Five: file ../../Keyboard/key.kicad_sch -> ../Keyboard/key.kicad_sch
- sheet Four: file ../../Keyboard/key.kicad_sch -> ../Keyboard/key.kicad_sch
- sheet Minus: file ../../Keyboard/key.kicad_sch -> ../Keyboard/key.kicad_sch
- sheet Nine: file ../../Keyboard/key.kicad_sch -> ../Keyboard/key.kicad_sch
- sheet Num: file ../../Keyboard/key.kicad_sch -> ../Keyboard/key.kicad_sch
- sheet One: file ../../Keyboard/key.kicad_sch -> ../Keyboard/key.kicad_sch
- sheet Over: file ../../Keyboard/key.kicad_sch -> ../Keyboard/key.kicad_sch
- sheet Plus: file ../../Keyboard/key.kicad_sch -> ../Keyboard/key.kicad_sch
- sheet Point: file ../../Keyboard/key.kicad_sch -> ../Keyboard/key.kicad_sch
- sheet Seven: file ../../Keyboard/key.kicad_sch -> ../Keyboard/key.kicad_sch
- sheet Six: file ../../Keyboard/key.kicad_sch -> ../Keyboard/key.kicad_sch
- sheet Three: file ../../Keyboard/key.kicad_sch -> ../Keyboard/key.kicad_sch
- sheet Times: file ../../Keyboard/key.kicad_sch -> ../Keyboard/key.kicad_sch
- sheet Two: file ../../Keyboard/key.kicad_sch -> ../Keyboard/key.kicad_sch
- sheet Zero: file ../../Keyboard/key.kicad_sch -> ../Keyboard/key.kicad_sch
Changed lines of the file:
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@@
 		(unit 1)
 		(exclude_from_sim no)
-		(in_bom yes)
+		(in_bom no)
 		(on_board yes)
 		(dnp no)
@@
 		)
 		(property "Description" "9-pin male plug pin D-SUB connector"
+			(at 262.89 62.23 0)
+			(effects
+				(font
+					(size 1.27 1.27)
+				)
+				(hide yes)
+			)
+		)
+		(property "JLCPCB Position Offset" ""
 			(at 262.89 62.23 0)
 			(effects
@@
 		(unit 1)
 		(exclude_from_sim no)
-		(in_bom yes)
+		(in_bom no)
 		(on_board yes)
 		(dnp no)
@@
 		)
 		(property "Description" "9-pin male plug pin D-SUB connector"
+			(at 262.89 97.79 0)
+			(effects
+				(font
+					(size 1.27 1.27)
+				)
+				(hide yes)
+			)
+		)
+		(property "JLCPCB Position Offset" ""
 			(at 262.89 97.79 0)
 			(effects
@@
 		(unit 1)
 		(exclude_from_sim no)
-		(in_bom yes)
+		(in_bom no)
 		(on_board yes)
 		(dnp no)
@@
 		)
 		(property "Description" "Push button switch, generic, two pins"
+			(at 171.45 35.56 0)
+			(effects
+				(font
+					(size 1.27 1.27)
+				)
+				(hide yes)
+			)
+		)
+		(property "JLCPCB Position Offset" ""
 			(at 171.45 35.56 0)
 			(effects
@@
 		(unit 1)
 		(exclude_from_sim no)
-		(in_bom yes)
+		(in_bom no)
 		(on_board yes)
 		(dnp no)
@@
 		)
 		(property "Description" "Generic connector, double row, 02x20, counter clockwise pin numbering scheme (similar to DIP package numbering), script generated (kicad-library-utils/schlib/autogen/connector/)"
+			(at 238.76 142.24 0)
+			(effects
+				(font
+					(size 1.27 1.27)
+				)
+				(hide yes)
+			)
+		)
+		(property "JLCPCB Position Offset" ""
 			(at 238.76 142.24 0)
 			(effects
@@
 			)
 		)
-		(property "Sheetfile" "../../Keyboard/key.kicad_sch"
+		(property "Sheetfile" "../Keyboard/key.kicad_sch"
 			(at 115.57 172.0346 0)
 			(effects
@@
 			)
 		)
-		(property "Sheetfile" "../../Keyboard/key.kicad_sch"
+		(property "Sheetfile" "../Keyboard/key.kicad_sch"
 			(at 53.34 131.3946 0)
 			(effects
@@
 			)
 		)
-		(property "Sheetfile" "../../Keyboard/key.kicad_sch"
+		(property "Sheetfile" "../Keyboard/key.kicad_sch"
 			(at 83.82 112.3446 0)
 			(effects
@@
 			)
 		)
-		(property "Sheetfile" "../../Keyboard/key.kicad_sch"
+		(property "Sheetfile" "../Keyboard/key.kicad_sch"
 			(at 83.82 131.3946 0)
 			(effects
@@
 			)
 		)
-		(property "Sheetfile" "../../Keyboard/key.kicad_sch"
+		(property "Sheetfile" "../Keyboard/key.kicad_sch"
 			(at 83.82 151.7146 0)
 			(effects
@@
 			)
 		)
-		(property "Sheetfile" "../../Keyboard/key.kicad_sch"
+		(property "Sheetfile" "../Keyboard/key.kicad_sch"
 			(at 115.57 112.3446 0)
 			(effects
@@
 			)
 		)
-		(property "Sheetfile" "../../Keyboard/key.kicad_sch"
+		(property "Sheetfile" "../Keyboard/key.kicad_sch"
 			(at 22.86 192.3546 0)
 			(effects
@@
 			)
 		)
-		(property "Sheetfile" "../../Keyboard/key.kicad_sch"
+		(property "Sheetfile" "../Keyboard/key.kicad_sch"
 			(at 53.34 151.7146 0)
 			(effects
@@
 			)
 		)
-		(property "Sheetfile" "../../Keyboard/key.kicad_sch"
+		(property "Sheetfile" "../Keyboard/key.kicad_sch"
 			(at 22.86 112.3446 0)
 			(effects
@@
 			)
 		)
-		(property "Sheetfile" "../../Keyboard/key.kicad_sch"
+		(property "Sheetfile" "../Keyboard/key.kicad_sch"
 			(at 22.86 151.7146 0)
 			(effects
@@
 			)
 		)
-		(property "Sheetfile" "../../Keyboard/key.kicad_sch"
+		(property "Sheetfile" "../Keyboard/key.kicad_sch"
 			(at 115.57 131.3946 0)
 			(effects
@@
 			)
 		)
-		(property "Sheetfile" "../../Keyboard/key.kicad_sch"
+		(property "Sheetfile" "../Keyboard/key.kicad_sch"
 			(at 83.82 192.3546 0)
 			(effects
@@
 			)
 		)
-		(property "Sheetfile" "../../Keyboard/key.kicad_sch"
+		(property "Sheetfile" "../Keyboard/key.kicad_sch"
 			(at 53.34 112.3446 0)
 			(effects
@@
 			)
 		)
-		(property "Sheetfile" "../../Keyboard/key.kicad_sch"
+		(property "Sheetfile" "../Keyboard/key.kicad_sch"
 			(at 22.86 172.0346 0)
 			(effects
@@
 			)
 		)
-		(property "Sheetfile" "../../Keyboard/key.kicad_sch"
+		(property "Sheetfile" "../Keyboard/key.kicad_sch"
 			(at 83.82 172.0346 0)
 			(effects
@@
 			)
 		)
-		(property "Sheetfile" "../../Keyboard/key.kicad_sch"
+		(property "Sheetfile" "../Keyboard/key.kicad_sch"
 			(at 22.86 131.3946 0)
 			(effects
@@
 			)
 		)
-		(property "Sheetfile" "../../Keyboard/key.kicad_sch"
+		(property "Sheetfile" "../Keyboard/key.kicad_sch"
 			(at 53.34 172.0346 0)
 			(effects

Commit message: DecenTKL NumPad rev. 1 finalized
Parts:
- SW1: footprint Button_Switch_THT:SW_Tactile_SPST_Angled_PTS645Vx83-2LFS -> DecenTKL:SW_Push_1P1T_XKB_TS-1177A-C; JLCPCB Part # (none) -> C883269; now in the parts list
Other:
- sheet Enter: file ../Keyboard/key.kicad_sch -> key_2Uv.kicad_sch
- sheet Plus: file ../Keyboard/key.kicad_sch -> key_2Uv.kicad_sch
- sheet Zero: file ../Keyboard/key.kicad_sch -> key_2U.kicad_sch
Changed lines of the file:
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@@
 		(unit 1)
 		(exclude_from_sim no)
-		(in_bom no)
+		(in_bom yes)
 		(on_board yes)
 		(dnp no)
@@
 			)
 		)
-		(property "Footprint" "Button_Switch_THT:SW_Tactile_SPST_Angled_PTS645Vx83-2LFS"
+		(property "Footprint" "DecenTKL:SW_Push_1P1T_XKB_TS-1177A-C"
 			(at 171.45 30.48 0)
 			(effects
@@
 		)
 		(property "JLCPCB Layer Override" ""
+			(at 171.45 35.56 0)
+			(effects
+				(font
+					(size 1.27 1.27)
+				)
+				(hide yes)
+			)
+		)
+		(property "JLCPCB Part #" "C883269"
 			(at 171.45 35.56 0)
 			(effects
@@
 			)
 		)
-		(property "Sheetfile" "../Keyboard/key.kicad_sch"
+		(property "Sheetfile" "key_2Uv.kicad_sch"
 			(at 115.57 172.0346 0)
 			(effects
@@
 			)
 		)
-		(property "Sheetfile" "../Keyboard/key.kicad_sch"
+		(property "Sheetfile" "key_2U.kicad_sch"
 			(at 22.86 192.3546 0)
 			(effects
@@
 			)
 		)
-		(property "Sheetfile" "../Keyboard/key.kicad_sch"
+		(property "Sheetfile" "key_2Uv.kicad_sch"
 			(at 115.57 131.3946 0)
 			(effects
