File: DecenTKL/NumPad/key_choc.kicad_sch (KiCad schematic)
At the start: 4 parts, among them SW17 SW_Push

Commit message: DecenTKL numpad
Parts:
- SW2: renamed from SW17; footprint DecenTKL:Kailh_socket_MX_1-00U -> DecenTKL:Kailh_socket_Choc_1-50U-XE
- renumbered C16 to C1, D31 to D1

Commit message: DecenTKL numpad update
Parts:
- C2: renamed from C1; value 104 -> 100nF; JLCPCB Part # C83054 -> C14663
- D32: footprint DecenTKL:SK6812 MINI-EA -> LED_SMD:LED_SK6812MINI_PLCC4_3.5x3.5mm_P1.75mm; symbol LED:SK6812MINI -> DecentUSB_Library:SK6812MINI
- SW3: renamed from SW2; footprint DecenTKL:Kailh_socket_Choc_1-50U-XE -> DecenTKL:Kailh_socket_MX_1-00U
- renumbered D1 to D3
Connections:
- net GND: now also D32.3 (VSS); no longer D32.2 (VSS)
- net RGB_IN: now also D32.4 (DIN); no longer D32.3 (DIN)
- net RGB_OUT: now also D32.2 (DOUT); no longer D32.1 (DOUT)
- net VBUS: now also D32.1 (VDD); no longer D32.4 (VDD)
Changed lines of the file:
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@@
 		(on_board yes)
 		(dnp no)
-		(fields_autoplaced yes)
-		(property "Reference" "D1"
-			(at 134.112 92.7678 90)
+		(property "Reference" "D3"
+			(at 133.858 94.234 90)
 			(effects
 				(font
@@
 		)
 		(property "Value" "1N4148W"
-			(at 134.112 95.1921 90)
+			(at 132.334 96.774 90)
 			(effects
 				(font
@@
 		)
 		(property "JLCPCB Rotation Offset" ""
+			(at 132.08 93.98 0)
+			(effects
+				(font
+					(size 1.27 1.27)
+				)
+				(hide yes)
+			)
+		)
+		(property "JLCPCB Position Offset" ""
 			(at 132.08 93.98 0)
 			(effects
@@
 		(dnp no)
 		(fields_autoplaced yes)
-		(property "Reference" "C1"
+		(property "Reference" "C2"
 			(at 181.991 94.0378 0)
 			(effects
@@
 			)
 		)
-		(property "Value" "104"
+		(property "Value" "100nF"
 			(at 181.991 96.4621 0)
 			(effects
@@
 			)
 		)
-		(property "JLCPCB Part #" " C83054"
+		(property "JLCPCB Part #" "C14663"
 			(at 179.07 95.25 0)
 			(effects
@@
 		)
 		(property "JLCPCB Rotation Offset" ""
+			(at 179.07 95.25 0)
+			(effects
+				(font
+					(size 1.27 1.27)
+				)
+				(hide yes)
+			)
+		)
+		(property "JLCPCB Position Offset" ""
 			(at 179.07 95.25 0)
 			(effects
@@
 		(dnp no)
 		(fields_autoplaced yes)
-		(property "Reference" "#PWR053"
+		(property "Reference" "#PWR054"
 			(at 179.07 109.22 0)
 			(effects
@@
 		(on_board yes)
 		(dnp no)
-		(fields_autoplaced yes)
-		(property "Reference" "SW2"
-			(at 127 90.7245 0)
+		(property "Reference" "SW3"
+			(at 127 93.726 0)
 			(effects
 				(font
@@
 		)
 		(property "Value" "SW_Push"
-			(at 127 93.1488 0)
-			(effects
-				(font
-					(size 1.27 1.27)
-				)
-			)
-		)
-		(property "Footprint" "DecenTKL:Kailh_socket_Choc_1-50U-XE"
+			(at 127 99.568 0)
+			(effects
+				(font
+					(size 1.27 1.27)
+				)
+			)
+		)
+		(property "Footprint" "DecenTKL:Kailh_socket_MX_1-00U"
 			(at 127 92.71 0)
 			(effects
@@
 		)
 		(property "JLCPCB Rotation Offset" ""
+			(at 127 97.79 0)
+			(effects
+				(font
+					(size 1.27 1.27)
+				)
+				(hide yes)
+			)
+		)
+		(property "JLCPCB Position Offset" ""
 			(at 127 97.79 0)
 			(effects
@@
 		(dnp no)
 		(fields_autoplaced yes)
-		(property "Reference" "#PWR075"
+		(property "Reference" "#PWR076"
 			(at 179.07 91.44 0)
 			(effects
@@
 	)
 	(symbol
-		(lib_id "LED:SK6812MINI")
+		(lib_id "DecentUSB_Library:SK6812MINI")
 		(at 157.48 95.25 0)
 		(unit 1)
@@
 			)
 		)
-		(property "Footprint" "DecenTKL:SK6812 MINI-EA"
+		(property "Footprint" "LED_SMD:LED_SK6812MINI_PLCC4_3.5x3.5mm_P1.75mm"
 			(at 158.75 102.87 0)
 			(effects
@@
 			(at 157.48 95.25 0)
 			(effects
+				(font
+					(size 1.27 1.27)
+				)
+				(hide yes)
+			)
+		)
+		(property "JLCPCB Position Offset" ""
+			(at 157.48 95.25 0)
+			(effects

Commit message: DecenTKL NumPad WIP
Parts:
- SW3: value SW_Push -> MX; JLCPCB Layer Override (none) -> B.Cu; JLCPCB Part # C5333465 -> C5156480
Changed lines of the file:
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@@
+			)
+		)
+		(property "JLCPCB Layer Override" ""
+			(at 132.08 93.98 0)
+			(effects
+				(font
+					(size 1.27 1.27)
+				)
+				(hide yes)
 			)
 		)
@@
 			)
 		)
+		(property "JLCPCB Layer Override" ""
+			(at 179.07 95.25 0)
+			(effects
+				(font
+					(size 1.27 1.27)
+				)
+				(hide yes)
+			)
+		)
 		(pin "1"
 		)
@@
 			)
 		)
-		(property "Value" "SW_Push"
+		(property "Value" "MX"
 			(at 127 99.568 0)
 			(effects
@@
 			)
 		)
-		(property "JLCPCB Part #" "C5333465"
+		(property "JLCPCB Part #" "C5156480"
 			(at 127 97.79 0)
 			(effects
@@
 		)
 		(property "JLCPCB Position Offset" ""
+			(at 127 97.79 0)
+			(effects
+				(font
+					(size 1.27 1.27)
+				)
+				(hide yes)
+			)
+		)
+		(property "JLCPCB Layer Override" "B.Cu"
 			(at 127 97.79 0)
 			(effects
@@
 			(at 157.48 95.25 0)
 			(effects
+				(font
+					(size 1.27 1.27)
+				)
+				(hide yes)
+			)
+		)
+		(property "JLCPCB Layer Override" ""
+			(at 157.48 95.25 0)
+			(effects

Commit message: DecenTKL NumPad rev. 1 finalized
Parts:
- SW3: value MX -> Choc; footprint DecenTKL:Kailh_socket_MX_1-00U -> DecenTKL:Kailh_socket_Choc_1-50U-XE; JLCPCB Part # C5156480 -> C5333465
Changed lines of the file:
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@@
 			)
 		)
-		(property "Value" "MX"
+		(property "Value" "Choc"
 			(at 127 99.568 0)
 			(effects
@@
 			)
 		)
-		(property "Footprint" "DecenTKL:Kailh_socket_MX_1-00U"
+		(property "Footprint" "DecenTKL:Kailh_socket_Choc_1-50U-XE"
 			(at 127 92.71 0)
 			(effects
@@
 			)
 		)
-		(property "JLCPCB Part #" "C5156480"
+		(property "JLCPCB Part #" "C5333465"
 			(at 127 97.79 0)
 			(effects
