File: misc-models/Atari/S-Video/S-Video.kicad_sch (KiCad schematic)
At the start: 40 parts, among them J1 GTIA, J2 Power, J3 Video out, Q1 NPN, Q2 NPN, U1 4050, U2 FMS6410B

Commit message: Atari S-video mod prototype
Parts:
- C1, C3, C4, C5: JLCPCB Part # (none) -> C1525
- C2: JLCPCB Part # (none) -> C32949
- C6: JLCPCB Part # (none) -> C15525
- C7: FT Rotation Offset (none) -> 180
- R1, R2, R22, R24, R3, R4, R5: JLCPCB Part # (none) -> C11702
- R10: JLCPCB Part # (none) -> C25762
- R11: JLCPCB Part # (none) -> C4908
- R12: JLCPCB Part # (none) -> C25077
- R13: JLCPCB Part # (none) -> C4109
- R14, R15, R16, R17, R18: JLCPCB Part # (none) -> C25133
- R19, R21, R8: JLCPCB Part # (none) -> C25900
- R20: JLCPCB Part # (none) -> C25744
- R23: JLCPCB Part # (none) -> C137946
- R6: JLCPCB Part # (none) -> C25132
- R7: JLCPCB Part # (none) -> C43676
- R9: JLCPCB Part # (none) -> C25926
