File: DecentCart/DecentCart2040/DecentCart2040.kicad_pcb (KiCad board)
At the start: 2 copper layers, 56 x 73 mm, 80 parts, among them J1 Micro_SD_Card, J2 Conn_02x15_Row_Letter_First, J3 SM03B-SRSS-TB, J7 Conn_01x04, J8 USB_B_Micro, J9 SM03B-SRSS-TB, Q2 TP0610L, SW2 SW_TACTILE, SW3 SW_TACTILE, U1 SN74LVC8T245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

Commit message: DecentCart 2040 rev. 1.1 fixes
Parts:
- added D3: MBR120VLSFT1G, Diode_SMD:Nexperia_CFP3_SOD-123W, F.Cu at (82.8, 70.9)
- Q2: value TP0610L -> DMG2305UX
- moved C26 2.60 mm to (79.7, 68.6)
- moved Q2 2.04 mm to (82.5, 74.2)
Connections:
- C18 pad 2: +5V -> +5V HOST
- C19 pad 2: +5V -> +5V HOST
- C2 pad 2: +5V -> +5V HOST
- C26 pad 1: VBUS -> Net-(D3-K)
- C3 pad 2: +5V -> +5V HOST
- C30 pad 2: +5V -> +5V HOST
- C31 pad 2: +5V -> +5V HOST
- C39 pad 2: +5V -> +5V HOST
- C40 pad 2: +5V -> +5V HOST
- J7 pad 3: GPIO28 -> GPIO29
- J7 pad 4: GPIO29 -> GPIO28
- J8 pad 1: VBUS -> /VBUS
- Q2 pad 1: +5V -> Net-(D3-K)
- Q2 pad 2: VBUS -> /VBUS
- U1 pad 23: +5V -> +5V HOST
- U1 pad 24: +5V -> +5V HOST
- U2 pad 23: +5V -> +5V HOST
- U2 pad 24: +5V -> +5V HOST
- U3 pad 13: GPIO29 -> GPIO28
- U3 pad 14: GPIO28 -> GPIO29
- U4 pad 3: VBUS -> Net-(D3-K)
- U5 pad 23: +5V -> +5V HOST
- U5 pad 24: +5V -> +5V HOST
- U6 pad 16: +5V -> +5V HOST
Routing:
- net +5V HOST: track 22.2 -> 116.0 mm, vias 0 -> 7
- net +5V: track 88.4 -> 0.00 mm, vias 6 -> 0
- net /VBUS: track 0.00 -> 87.5 mm, vias 0 -> 4
- net VBUS: track 82.8 -> 0.00 mm, vias 2 -> 0
- net GND: track 379.2 -> 389.7 mm, vias 58 -> 55
- net Net-(D3-K): track 0.00 -> 8.08 mm
- net GPIO28: track 32.3 -> 39.9 mm
- net GPIO29: track 35.1 -> 33.8 mm, vias 1 -> 2
- net RD5: track 34.3 -> 33.0 mm
Other:
- board text added: "AtTiny flash"
- board text added: "RP2040 debug"

Commit message: DecentCart2040 rev. 1.1
Parts:
- added C15: 100nF, Capacitor_SMD:C_0402_1005Metric, F.Cu at (67.1, 71.1)
- added C20: 100nF, Capacitor_SMD:C_0402_1005Metric, F.Cu at (70.2, 71.1)
- added C21: 1uF, Capacitor_SMD:C_0402_1005Metric, F.Cu at (69.2, 71.1)
- added J4: Conn_01x08_Pin, Connector_PinHeader_1.27mm:PinHeader_2x04_P1.27mm_Vertical, F.Cu at (82.0, 46.4)
- added U8: SN74LVC2T45DCUR, Package_SO:VSSOP-8_2.3x2mm_P0.5mm, F.Cu at (68.9, 73.4)
- U6: value SN74AVC4T245PW -> SN74LVC2T45DCUR; footprint Package_SO:TSSOP-16_4.4x5mm_P0.65mm -> Package_SO:VSSOP-8_2.3x2mm_P0.5mm
- moved C40 12.5 mm to (63.8, 74.7), turned to -90 degrees
- moved C39 11.2 mm to (64.8, 74.7), turned to -90 degrees
- moved R3 10.8 mm to (73.4, 72.7), turned to 180 degrees
- moved U6 9.44 mm to (61.5, 75.6), turned to -45 degrees
- moved R2 7.84 mm to (63.7, 78.2), turned to 180 degrees
- moved C38 4.76 mm to (61.8, 72.7), turned to -135 degrees
- moved R10 4.05 mm to (68.9, 32.5)
- moved C31 3.33 mm to (75.2, 82.7), turned to 180 degrees
- moved C30 1.94 mm to (75.2, 83.6), turned to 180 degrees
- moved R11 0.99 mm to (87.8, 57.1)
Connections:
- D2 pad 1: Net-(D2-K) -> Net-(D1-A)
- J1 pad 9: unconnected-(J1-DET-Pad9) -> Net-(J1-DET)
- J3 pad 1: +3V3 -> Net-(J3-Pin_1)
- J3 pad 2: GND -> +3V3
- J3 pad 3: Net-(J3-Pin_3) -> GND
- R1 pad 1: R/W -> GPIO23
- R10 pad 1: Net-(U3-PB2) -> Net-(U3-PA6)
- R10 pad 2: Net-(D1-A) -> Net-(D1-K)
- R2 pad 2: Net-(U6-2DIR) -> Net-(U6-DIR)
- R3 pad 2: Net-(U6-1DIR) -> Net-(U8-DIR)
- U3 pad 10: unconnected-(U3-PB4-Pad10) -> Net-(J4-Pin_7)
- U3 pad 11: Net-(D2-K) -> Net-(J4-Pin_6)
- U3 pad 12: Net-(U3-PB2) -> Net-(J4-Pin_5)
- U3 pad 15: unconnected-(U3-PC0-Pad15) -> Net-(J4-Pin_1)
- U3 pad 16: unconnected-(U3-PC1-Pad16) -> Net-(J4-Pin_2)
- U3 pad 17: unconnected-(U3-PC2-Pad17) -> Net-(J4-Pin_3)
- U3 pad 18: unconnected-(U3-PC3-Pad18) -> Net-(J4-Pin_4)
- U3 pad 19: Net-(J3-Pin_3) -> Net-(J3-Pin_1)
- U3 pad 6: unconnected-(U3-PA5-Pad6) -> Net-(J1-DET)
- U3 pad 7: unconnected-(U3-PA6-Pad7) -> Net-(U3-PA6)
- U3 pad 8: unconnected-(U3-PA7-Pad8) -> Net-(D1-A)
- U6 pad 2: Net-(U6-1DIR) -> GPIO24
- U6 pad 3: Net-(U6-2DIR) -> GPIO25
- U6 pad 4: GPIO26 -> GND
- U6 pad 5: GPIO27 -> Net-(U6-DIR)
- U6 pad 6: GPIO24 -> /S5
- U6 pad 7: GPIO25 -> /S4
- U6 pad 8: GND -> +5V HOST
Routing:
- net Net-(D1-A): track 4.45 -> 54.5 mm, vias 0 -> 2
- net Net-(U3-PA6): track 0.00 -> 44.7 mm, vias 0 -> 2
- net Net-(D2-K): track 34.1 -> 0.00 mm
- net Net-(U3-PB2): track 26.9 -> 0.00 mm
- net R/W: track 41.3 -> 16.5 mm, vias 3 -> 1
- net Net-(J4-Pin_7): track 0.00 -> 22.2 mm, vias 0 -> 1
- net +3V3: track 226.6 -> 247.4 mm, vias 12 -> 14
- net Net-(J3-Pin_1): track 0.00 -> 19.1 mm, vias 0 -> 2
- net Net-(J1-DET): track 0.00 -> 18.1 mm, vias 0 -> 2
- net Net-(J3-Pin_3): track 18.0 -> 0.00 mm, vias 2 -> 0
- net GPIO23: track 40.0 -> 55.6 mm, vias 2 -> 4
- net /S5: track 28.1 -> 40.4 mm
- net Net-(J4-Pin_1): track 0.00 -> 11.0 mm, vias 0 -> 2
- net /S4: track 49.1 -> 38.9 mm
- net Net-(J4-Pin_5): track 0.00 -> 8.99 mm
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Other:
- board text added: "3V3"
- board text added: "GND"
- board text added: "SWCLK"
- board text added: "SWD"
- board text added: "UPDI"
