File: DecentCart/DecentCart.kicad_pcb (KiCad board)
At the start: 2 copper layers, 76 parts, among them J1 Micro_SD_Card, J2 Conn_02x15_Row_Letter_First, J3 Conn_02x07_Row_Letter_First, J7 Conn_01x08, J8 USB_B_Micro, J9 SM03B-SRSS-TB, Q2 TP0610L, SW1 RotaryEncoder_Switch_MP, SW2 SW_USB_BOOT, SW3 SW_RESET, U1 SN74LVC8T245, U2 SN74LVC8T245, U3 RP2350_80QFN, U4 NCP1117-3.3_SOT223, U5 SN74LVC8T245, U6 SN74LVC8T245, U8 SN74LVC8T245, U9 W25Q128JVS, X1 12MHz

Commit message: DecentCart 2350 component placement
Parts:
- removed SW1: RotaryEncoder_Switch_MP, DecenTKL:Thin Side Encoder
- added D1: MBR120VLSFT1G, Diode_SMD:Nexperia_CFP3_SOD-123W, F.Cu at (134.8, 61.3)
- added G***: LOGO, Library:ScreamingAtTheRadio, F.Cu at (126.7, 77.5)
- added G***: LOGO, Library:ScreamingAtTheRadio, B.Cu at (152.3, 61.2)
- added H1: MountingHole, MountingHole:MountingHole_2.2mm_M2, F.Cu at (149.8, 73.5)
- added H2: MountingHole, MountingHole:MountingHole_2.2mm_M2, F.Cu at (174.3, 95.5)
- added H3: MountingHole, MountingHole:MountingHole_2.2mm_M2, F.Cu at (125.5, 95.5)
- added J5: Conn_01x04_MountingPin, Connector_JST:JST_SH_SM04B-SRSS-TB_1x04-1MP_P1.00mm_Horizontal, F.Cu at (177.7, 81.9)
- added R10: 1k, Resistor_SMD:R_0402_1005Metric, F.Cu at (138.6, 91.1)
- added R2: 1k, Resistor_SMD:R_0402_1005Metric, F.Cu at (158.2, 93.4)
- added R3: 1k, Resistor_SMD:R_0402_1005Metric, F.Cu at (144.7, 97.2)
- added REF**: KiCad-Logo2_6mm_Copper, Symbol:KiCad-Logo2_6mm_Copper, F.Cu at (126.0, 59.6)
- added REF**: OSHW-Logo2_7.3x6mm_Copper, Symbol:OSHW-Logo2_7.3x6mm_Copper, F.Cu at (125.0, 69.3)
- added REF**: KiCad-Logo2_6mm_Copper, Symbol:KiCad-Logo2_6mm_Copper, B.Cu at (170.6, 61.7)
- added REF**: OSHW-Logo2_7.3x6mm_Copper, Symbol:OSHW-Logo2_7.3x6mm_Copper, B.Cu at (160.6, 62.8)
- C10, C11, C12, C13, C14, C15, C4, C42, C6, C7, C8, C9: value 100n -> 100nF
- C20, C21, C22, C5: value 4.7u -> 4.7uF
- C26, C27, C28: value 10u -> 10uF
- J3: footprint Connector_PinSocket_2.54mm:PinSocket_2x07_P2.54mm_Horizontal -> Connector_PinSocket_2.54mm:PinSocket_2x07_P2.54mm_Vertical
- L16: value 3.3u -> 3.3uH
- Q2: value TP0610L -> DMG2305UX
- R37: footprint Resistor_SMD:R_0402_1005Metric -> Jumper:SolderJumper-2_P1.3mm_Bridged_RoundedPad1.0x1.5mm
- SW2: value SW_USB_BOOT -> SW_TACTILE; footprint DecenTKL:SW_Push_1P1T_XKB_TS-1177A-C -> DecenTKL:Tactile_Switch_Basic_XKB_TS-1187A
- SW3: value SW_RESET -> SW_TACTILE; footprint DecenTKL:SW_Push_1P1T_XKB_TS-1177A-C -> DecenTKL:Tactile_Switch_Basic_XKB_TS-1187A
- moved J1 221.9 mm to (167.5, 57.3), turned to 180 degrees
- moved C16 210.0 mm to (169.1, 70.1), turned to 90 degrees
- moved C23 206.1 mm to (168.2, 70.1), turned to 90 degrees
- moved C39 205.3 mm to (171.2, 94.6), turned to 45 degrees
- moved C40 204.3 mm to (170.5, 93.9), turned to 45 degrees
- moved J2 203.4 mm to (132.0, 119.8)
- moved C33 201.6 mm to (165.7, 99.5), turned to 135 degrees
- moved C34 200.7 mm to (165.0, 100.2), turned to 135 degrees
- moved C5 200.1 mm to (155.5, 88.3), turned to -45 degrees
- moved C38 200.1 mm to (166.7, 87.0), turned to -45 degrees
- moved C11 198.2 mm to (156.6, 81.9), turned to 45 degrees
- moved C4 198.2 mm to (154.1, 79.3), turned to 45 degrees
- moved U5 197.0 mm to (149.5, 103.0), turned to -90 degrees
- moved U6 196.8 mm to (159.7, 98.7), turned to -45 degrees
- moved C10 196.3 mm to (154.7, 80.0), turned to 45 degrees
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Connections:
- C26 pad 1: VBUS -> Net-(D1-K)
- J1 pad 9: unconnected-(J1-DET-Pad9) -> GPIO39
- J2 pad 1: GPIO27 -> (no net)
- J2 pad 12: GPIO28 -> (no net)
- J2 pad 14: GPIO33 -> (no net)
- J2 pad 15: GPIO24 -> (no net)
- J2 pad A: GPIO32 -> (no net)
- J2 pad R: GPIO26 -> (no net)
- J2 pad S: GPIO25 -> (no net)
- J3 pad 1: GPIO35 -> /EXTSEL
- J3 pad 2: GPIO31 -> /RST
- J3 pad 4: GPIO36 -> /MPD
- J3 pad 6: GPIO30 -> REF
- J8 pad 1: VBUS -> /VBUS
- Q2 pad 1: +5V -> Net-(D1-K)
- Q2 pad 2: VBUS -> /VBUS
- R1 pad 1: GPIO26 -> R/W
- U1 pad 10: A7 -> GPIO0
- U1 pad 14: A7 -> A0
- U1 pad 15: A6 -> A1
- U1 pad 16: A5 -> A2
- U1 pad 17: A4 -> A3
- U1 pad 18: A3 -> A4
- U1 pad 19: A2 -> A5
- U1 pad 2: GND -> Net-(U1-DIR)
- U1 pad 20: A1 -> A6
- U1 pad 21: A0 -> A7
- U1 pad 3: A0 -> GPIO7
- U1 pad 4: A1 -> GPIO6
- U1 pad 5: A2 -> GPIO5
- U1 pad 6: A3 -> GPIO4
- U1 pad 7: A4 -> GPIO3
- U1 pad 8: A5 -> GPIO2
- U1 pad 9: A6 -> GPIO1
- U2 pad 10: A15 -> GPIO8
- U2 pad 14: A15 -> A8
- U2 pad 15: A14 -> A9
- U2 pad 16: A13 -> A10
- U2 pad 17: A12 -> A11
- U2 pad 18: A11 -> A12
- U2 pad 19: A10 -> A13
- U2 pad 2: GND -> Net-(U2-DIR)
- U2 pad 20: A9 -> A14
- U2 pad 21: A8 -> A15
- U2 pad 3: A8 -> GPIO15
- U2 pad 4: A9 -> GPIO14
- U2 pad 5: A10 -> GPIO13
- U2 pad 6: A11 -> GPIO12
- U2 pad 7: A12 -> GPIO11
- U2 pad 8: A13 -> GPIO10
- U2 pad 9: A14 -> GPIO9
- U3 pad 1: A4 -> GPIO4
- U3 pad 11: A12 -> GPIO12
- U3 pad 12: A13 -> GPIO13
- U3 pad 13: A14 -> GPIO14
- U3 pad 14: A15 -> GPIO15
- U3 pad 16: D0 -> GPIO16
- U3 pad 17: D1 -> GPIO17
- U3 pad 18: D2 -> GPIO18
- U3 pad 19: D3 -> GPIO19
- U3 pad 2: A5 -> GPIO5
- U3 pad 20: D4 -> GPIO20
- U3 pad 21: D5 -> GPIO21
- U3 pad 22: D6 -> GPIO22
- U3 pad 23: D7 -> GPIO23
- U3 pad 3: A6 -> GPIO6
- U3 pad 4: A7 -> GPIO7
- U3 pad 46: D1xx -> GPIO37
- U3 pad 6: A8 -> GPIO8
- U3 pad 7: A9 -> GPIO9
- U3 pad 77: A0 -> GPIO0
- U3 pad 78: A1 -> GPIO1
- U3 pad 79: A2 -> GPIO2
- U3 pad 8: A10 -> GPIO10
- U3 pad 80: A3 -> GPIO3
- U3 pad 9: A11 -> GPIO11
- U4 pad 3: VBUS -> Net-(D1-K)
- U5 pad 10: D7 -> GPIO16
- U5 pad 14: D7 -> D0
- U5 pad 15: D6 -> D1
- U5 pad 16: D5 -> D2
- U5 pad 17: D4 -> D3
- U5 pad 18: D3 -> D4
- U5 pad 19: D2 -> D5
- U5 pad 20: D1 -> D6
- U5 pad 21: D0 -> D7
- U5 pad 3: D0 -> GPIO23
- U5 pad 4: D1 -> GPIO22
- U5 pad 5: D2 -> GPIO21
- U5 pad 6: D3 -> GPIO20
- U5 pad 7: D4 -> GPIO19
- U5 pad 8: D5 -> GPIO18
- U5 pad 9: D6 -> GPIO17
- U6 pad 10: GPIO31 -> GPIO24
- U6 pad 14: GPIO31 -> /CCTL
- U6 pad 15: GPIO30 -> Phi2
- U6 pad 16: /HALT -> R/W
- U6 pad 17: GPIO28 -> /S4
- U6 pad 18: GPIO27 -> /S5
- U6 pad 19: GPIO26 -> /HALT
- U6 pad 2: GND -> Net-(U6-DIR)
- U6 pad 20: GPIO25 -> REF
- U6 pad 21: GPIO24 -> /RST
- U6 pad 3: GPIO24 -> GPIO31
- U6 pad 4: GPIO25 -> GPIO30
- U6 pad 5: GPIO26 -> GPIO29
- U6 pad 6: GPIO27 -> GPIO28
- U6 pad 7: GPIO28 -> GPIO27
- U6 pad 8: GPIO29 -> GPIO26
- U6 pad 9: GPIO30 -> GPIO25
- U8 pad 16: D1xx -> RD4
- U8 pad 17: GPIO36 -> RD5
- U8 pad 18: GPIO35 -> /IRQ
- U8 pad 19: GPIO34 -> /EXTSEL
- U8 pad 20: GPIO33 -> /MPD
- U8 pad 21: GPIO32 -> D1xx
- U8 pad 3: GPIO32 -> GPIO37
- U8 pad 4: GPIO33 -> GPIO36
- U8 pad 5: GPIO34 -> GPIO35
- U8 pad 6: GPIO35 -> GPIO34
- U8 pad 7: GPIO36 -> GPIO33
- U8 pad 8: D1xx -> GPIO32
Routing:
- added copper zone on B.Cu, net GND
- added copper zone on F.Cu, net GND
Other:
- board outline added: 59.3 x 73 mm
- board text added: "DecentCart 2350"
- board text added: "Rev. 1"
- board text added: "https://github.com/bleroy/3d-junkyard/tree/main/DecentCart"
- board text added: "©Bertrand Le Roy 2025"

Commit message: DecenttCart 2350 routed
Parts:
- J3: value Conn_02x07_Row_Letter_First -> QWIIC / Stemma I2C
- J8: footprint Connector_USB:USB_Micro-B_Amphenol_10103594-0001LF_Horizontal -> Library:USB_Micro-B
- J9: value SM03B-SRSS-TB -> Debug
- R26, R28: footprint Resistor_SMD:R_0402_1005Metric -> Resistor_SMD:R_0805_2012Metric
- ST7789 SPI Display: renamed from J7; moved to B.Cu
- U3: value RP2350_80QFN -> RP2350B
- U9: footprint Package_SO:SOIC-8_7.5x5.85mm_P1.27mm -> Package_SO:SOIC-8_5.23x5.23mm_P1.27mm
- moved H3 48.8 mm to (174.3, 94.3)
- moved H2 33.8 mm to (149.8, 72.3)
- moved H1 31.9 mm to (125.5, 94.3)
- moved R32 11.7 mm to (157.8, 65.4)
- moved C22 10.1 mm to (155.4, 73.5), turned to -45 degrees
- moved C21 7.78 mm to (154.8, 74.1), turned to -45 degrees
- moved L16 7.54 mm to (153.6, 73.0), turned to -135 degrees
- moved R25 5.93 mm to (154.1, 74.8), turned to 135 degrees
- moved R37 4.80 mm to (136.2, 72.5), turned to -135 degrees
- moved SW3 4.69 mm to (154.3, 54.2), turned to 180 degrees
- moved U9 2.75 mm to (141.3, 73.4)
- moved R28 2.66 mm to (146.0, 75.6)
- moved C20 2.55 mm to (153.4, 75.5), turned to -45 degrees
- moved R26 2.30 mm to (144.6, 77.0)
- moved R30 1.52 mm to (146.0, 56.6)
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Connections:
- J2 pad 1: (no net) -> /S4
- J2 pad 12: (no net) -> /S5
- J2 pad 13: +5V HOST -> +5V
- J2 pad 14: (no net) -> RD5
- J2 pad 15: (no net) -> /CCTL
- J2 pad A: (no net) -> RD4
- J2 pad R: (no net) -> R/W
- J2 pad S: (no net) -> Phi2
- J3 pad 7: +5V HOST -> +5V
- Q2 pad 3: +5V HOST -> +5V
Routing:
- net GND: track 0.00 -> 558.4 mm, vias 0 -> 43
- net +3V3: track 0.00 -> 250.0 mm, vias 0 -> 7
- net +5V: track 0.00 -> 161.4 mm, vias 0 -> 4
- net GPIO38: track 0.00 -> 82.1 mm, vias 0 -> 4
- net RD4: track 0.00 -> 71.3 mm, vias 0 -> 1
- net /S4: track 0.00 -> 61.9 mm, vias 0 -> 2
- net A15: track 0.00 -> 52.4 mm
- net A13: track 0.00 -> 51.8 mm
- net A14: track 0.00 -> 51.6 mm
- net GPIO42: track 0.00 -> 48.9 mm, vias 0 -> 1
- net A3: track 0.00 -> 43.7 mm
- net GPIO43: track 0.00 -> 43.6 mm, vias 0 -> 1
- net SPI TX: track 0.00 -> 41.2 mm, vias 0 -> 2
- net A11: track 0.00 -> 40.9 mm, vias 0 -> 1
- net A2: track 0.00 -> 40.9 mm
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Other:
- board text added: "/CCTL"
- board text added: "/ExtSel"
- board text added: "/HLT"
- board text added: "/IRQ"
- board text added: "/MPD"
- board text added: "/RST"
- board text added: "/S4"
- board text added: "/S5"
- board text added: "3V3"
- board text added: "5V"
- board text added: "A13"
- board text added: "A14"
- board text added: "A15"
- board text added: "Aud"
- board text added: "Bullet Time"
- board text added: "CLK"
- board text added: "D1xx"
- board text added: "GND"
- board text added: "Phi2"
- board text added: "R/W"
- board text added: "RD4"
- board text added: "RD5"
- board text added: "REF"
- board text added: "Ref"
- board text added: "Res"
- board text added: "SCL"
- board text added: "SDA"
- board text added: "SWD"
- board text removed: "DecentCart 2350"

Commit message: BulletTime adjustments
Parts:
- moved REF** 13.1 mm to (158.9, 54.7)
- moved REF** 12.3 mm to (149.8, 55.8)
- moved G*** 12.3 mm to (141.7, 53.9)
Routing:
- net GND: track 558.4 -> 559.1 mm
Other:
- board text added: "A0"
- board text added: "A1"
- board text added: "A10"
- board text added: "A11"
- board text added: "A12"
- board text added: "A2"
- board text added: "A3"
- board text added: "A4"
- board text added: "A5"
- board text added: "A6"
- board text added: "A7"
- board text added: "A8"
- board text added: "A9"
- board text added: "BLK"
- board text added: "CS"
- board text added: "D0"
- board text added: "D1"
- board text added: "D2"
- board text added: "D3"
- board text added: "D4"
- board text added: "D5"
- board text added: "D6"
- board text added: "D7"
- board text added: "DC"
- board text added: "RES"
- board text added: "VCC"

Commit message: Small DecentCart2040 and 2350 changes
Parts:
- J3: value QWIIC / Stemma I2C -> Conn_02x07_Row_Letter_First
- J7: renamed from ST7789 SPI Display
- J9: value Debug -> SM03B-SRSS-TB
- U3: value RP2350B -> RP2350_80QFN
Other:
- board text added: "Debug"
- board text added: "QWIIC Stemma I2C ext."
- board text added: "ST7789 SPI display"

Commit message: DecentCart2350 Bullet Time rev.2
Parts:
- removed J5: Conn_01x04_MountingPin, Connector_JST:JST_SH_SM04B-SRSS-TB_1x04-1MP_P1.00mm_Horizontal
- added D2: LED, Diode_SMD:D_0805_2012Metric, F.Cu at (177.4, 52.5)
- added Q1: PNP, Package_TO_SOT_SMD:SOT-23, F.Cu at (176.7, 55.2)
- added R34: 220, Resistor_SMD:R_0402_1005Metric, F.Cu at (179.6, 53.0)
- L16: footprint Inductor_SMD:L_0603_1608Metric -> Library:L_0806_2016Metric
- moved C22 8.80 mm to (147.0, 75.9), turned to 45 degrees
- moved L16 7.84 mm to (146.0, 74.9), turned to 45 degrees
- moved C21 7.55 mm to (147.6, 76.6), turned to 45 degrees
- moved C42 6.86 mm to (137.3, 70.1), turned to -135 degrees
- moved R25 6.54 mm to (147.8, 73.1), turned to -45 degrees
- moved C20 4.44 mm to (149.1, 74.4)
- moved R37 3.99 mm to (132.5, 73.9)
- moved U9 3.99 mm to (137.6, 74.7)
- moved R26 2.84 mm to (141.8, 77.3)
- moved R28 2.84 mm to (143.2, 76.0)
- moved H2 2.70 mm to (149.8, 69.6)
- moved R36 1.69 mm to (132.2, 77.4)
- moved C27 0.94 mm to (140.0, 67.1)
- moved C26 0.90 mm to (145.0, 65.8)
- moved U4 0.89 mm to (140.9, 62.2)
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Connections:
- net GPIO39 renamed SD_DETECT
- net GPIO43 renamed DISP_CS
- net GPIO45 renamed SD_CS
- net Net-(U3-USB_DM) renamed /USB-
- net Net-(U3-USB_DP) renamed /USB+
- J7 pad 5: unconnected-(J7-Pin_5-Pad5) -> DISP_RST
- J7 pad 6: GPIO42 -> DISP_CMD
- R1 pad 1: R/W -> DATA_DIR
- U1 pad 22: GPIO38 -> SHIFT_ENABLE
- U2 pad 22: GPIO38 -> SHIFT_ENABLE
- U3 pad 47: GPIO38 -> SHIFT_ENABLE
- U3 pad 49: GPIO40 -> DISP_RST
- U3 pad 52: GPIO41 -> DISP_CMD
- U3 pad 53: GPIO42 -> DATA_DIR
- U5 pad 22: GPIO38 -> SHIFT_ENABLE
- U6 pad 22: GPIO38 -> SHIFT_ENABLE
- U8 pad 22: GPIO38 -> SHIFT_ENABLE
Routing:
- net GPIO38: track 82.1 -> 0.00 mm, vias 4 -> 0
- net SHIFT_ENABLE: track 0.00 -> 82.0 mm, vias 0 -> 4
- net DISP_CMD: track 0.00 -> 49.4 mm, vias 0 -> 1
- net GPIO42: track 48.9 -> 0.00 mm, vias 1 -> 0
- net DISP_RST: track 0.00 -> 40.4 mm, vias 0 -> 1
- net GPIO40: track 39.8 -> 0.00 mm, vias 2 -> 0
- net GPIO41: track 34.7 -> 0.00 mm, vias 2 -> 0
- net SD_CS: track 20.5 -> 45.3 mm, vias 2 -> 3
- net DATA_DIR: track 0.00 -> 19.9 mm, vias 0 -> 2
- net R/W: track 35.2 -> 24.2 mm, vias 3 -> 1
- net +3V3: track 250.0 -> 257.7 mm, vias 7 -> 5
- net /QSPI_SS: track 31.9 -> 39.2 mm
- net /FLASH_SS: track 7.37 -> 3.87 mm
- net GND: track 559.1 -> 562.3 mm, vias 43 -> 45
- net /VREG_LX: track 7.00 -> 3.96 mm
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Other:
- board text added: "DecentCart2350 Bullet Time"
- board text added: "Rev. 2"
- board text removed: "3V3"
- board text removed: "Bullet Time"
- board text removed: "QWIIC Stemma I2C ext."
- board text removed: "Rev. 1"
