File: DecentXE/Plate/DecentXE-plate-modern.kicad_pcb (KiCad board)
At the start: 2 copper layers, 289.2 x 99.3 mm, 97 parts, among them SW0 SW_Push_45deg, SW1 SW_Push_45deg, SW2 SW_Push_45deg, SW3 SW_Push_45deg, SW4 SW_Push_45deg, SW5 SW_Push_45deg, SW6 SW_Push_45deg, SW7 SW_Push_45deg, SW8 SW_Push_45deg, SW9 SW_Push_45deg

Commit message: DecentXE rev 16
[x] Power LED switched to red in BOM
[x] Optional red LED diffuser 3D model
[x] Mid-keyboard support 3D model
[x] Back of the board padding 3D model for better fit in the XE case
[x] Console keys have stabilization holes in PCB and plate
[x] Plate covers the whole width of the keyboard and conoles keys area
[x] PCB made 1.75mm deeper to reach the case's fins on the back of the keyboard area
[x] Remove legends from plate front so it's a uniform black between key caps
Parts:
- removed the G*** at (238.0, 129.2)
- removed the G*** at (145.8, 129.2)
- removed the G*** at (203.0, 129.2)
- removed the G*** at (288.7, 94.1)
- removed the G*** at (79.1, 110.1)
- removed the G*** at (226.8, 91.1)
- removed the G*** at (131.5, 91.1)
- removed the G*** at (269.6, 94.1)
- removed the G*** at (126.7, 129.2)
- removed the G*** at (283.9, 75.1)
- removed the G*** at (207.7, 91.1)
- removed the G*** at (212.2, 135.4)
- removed the G*** at (74.4, 91.1)
- removed the G*** at (98.2, 110.2)
- removed the G*** at (312.5, 113.2)
- removed the G*** at (212.5, 110.2)
- removed the G*** at (188.6, 91.1)
- removed the G*** at (150.6, 91.1)
- removed the G*** at (257.1, 129.2)
- removed the G*** at (88.6, 129.2)
- removed the G*** at (117.2, 110.1)
- removed the G*** at (93.4, 91.1)
- removed the G*** at (107.7, 129.2)
- removed the G*** at (183.9, 129.2)
- removed the G*** at (164.8, 129.2)
- removed the G*** at (174.4, 110.1)
- removed the G*** at (112.5, 91.1)
- removed the G*** at (155.3, 110.1)
- removed the G*** at (169.6, 91.1)
- removed the G*** at (136.3, 110.2)
- removed the G*** at (245.8, 91.1)
- removed the G*** at (266.6, 110.2)
- removed the G*** at (264.9, 75.1)
- removed the G*** at (231.5, 110.2)
- removed the G*** at (193.4, 110.1)
- removed the REF** at (328.8, 55.1)
- removed the REF** at (45.1, 55.1)
- added G***: Decent XE Logo, Library:Decent XE Logo, F.Cu at (42.8, 25.1)
- added SWFn1: SW_Push_45deg, Library:Choc-1-50U-Atari-Fn-Hole, F.Cu at (97.1, 32.6)
- added SWFn2: SW_Push_45deg, Library:Choc-1-50U-Atari-Fn-Hole, F.Cu at (125.7, 32.6)
- added SWFn3: SW_Push_45deg, Library:Choc-1-50U-Atari-Fn-Hole, F.Cu at (154.3, 32.6)
- added SWFn4: SW_Push_45deg, Library:Choc-1-50U-Atari-Fn-Hole, F.Cu at (182.8, 32.6)
- added SWHlp1: SW_Push_45deg, Library:Choc-1-50U-Atari-Fn-Hole, F.Cu at (211.4, 32.6)
- added SWOption1: SW_Push_45deg, Library:Choc-1-50U-Atari-Fn-Hole, F.Cu at (297.2, 32.6)
- added SWReset1: SW_Push_45deg, Library:Choc-1-50U-Atari-Fn-Hole, F.Cu at (325.7, 32.6)
- added SWSelect1: SW_Push_45deg, Library:Choc-1-50U-Atari-Fn-Hole, F.Cu at (268.6, 32.6)
- added SWStart1: SW_Push_45deg, Library:Choc-1-50U-Atari-Fn-Hole, F.Cu at (240.0, 32.6)
- moved G*** 150.5 mm to (33.8, 43.1)
- moved REF** 141.1 mm to (53.1, 41.4)
- moved REF** 140.0 mm to (66.8, 43.1)
Routing:
- removed copper zone on F.Cu, net GND
Other:
- board size 289.2 x 99.3 mm -> 329.2 x 131.1 mm
- board text added: "Decent XE Keyboard rev. 16m © Bertrand Le Roy 2026 github.com/bleroy/3d-junkyard/tree/main/DecentXE atariage.com/forums/profile/76850-screamingattheradio/ twitch.tv/screamingattheradio youtube.com/@ScreamingAtTheRadio"
- board text removed: "!"
- board text removed: "#"
- board text removed: "$"
- board text removed: "%"
- board text removed: "&"
- board text removed: "'"
- board text removed: "("
- board text removed: ")"
- board text removed: "*"
- board text removed: "+"
- board text removed: ","
- board text removed: "-"
- board text removed: "."
- board text removed: "/"
- board text removed: "0"
- board text removed: "1"
- board text removed: "2"
- board text removed: "3"
- board text removed: "4"
- board text removed: "5"
- board text removed: "6"
- board text removed: "7"
- board text removed: "8"
- board text removed: "9"
- board text removed: ":"
- board text removed: ";"
- board text removed: "<"
- board text removed: "="
- board text removed: ">"
- board text removed: "?"
- board text removed: "@"
- board text removed: "A"
- board text removed: "B"
- board text removed: "Break"
- board text removed: "C"
- board text removed: "Caps"
- board text removed: "Clear"
- board text removed: "Clr"
- board text removed: "Control"
- board text removed: "D"
- board text removed: "Del"
- board text removed: "E"
- board text removed: "Esc"
- board text removed: "F"
- board text removed: "G"
- board text removed: "H"
- board text removed: "I"
- board text removed: "Insert"
- board text removed: "J"
- board text removed: "K"
- board text removed: "Keyboard plate rev. 15m (c) Bertrand Le Roy 2023 twitch.tv/screamingattheradio youtube.com/@ScreamingAtTheRadio atariage.com/forums/profile/76850-screamingattheradio github.com/bleroy/3d-junkyard/tree/main/Atari130MX"
- board text removed: "L"
- board text removed: "M"
- board text removed: "N"
- board text removed: "O"
- board text removed: "P"
- board text removed: "Q"
- board text removed: "R"
- board text removed: "Return"
- board text removed: "S"
- board text removed: "Set"
- board text removed: "Shift"
- board text removed: "Space"
- board text removed: "T"
- board text removed: "Tab"
- board text removed: "U"
- board text removed: "V"
- board text removed: "W"
- board text removed: "X"
- board text removed: "Y"
- board text removed: "Z"
- board text removed: "["
- board text removed: "\"
- board text removed: "]"
- board text removed: "^"
- board text removed: "_"
- board text removed: "{dblquote}"
- board text removed: "|"
