File: DecentXE/Keyboard/DecentXE-Modern.kicad_sch (KiCad schematic)
At the start: 199 parts, among them J1 Conn_02x12_Odd_Even, J2 Conn_01x26, J3 Conn_01x04, SW0 SW_Push_45deg, SW1 SW_Push_45deg, SW2 SW_Push_45deg, SW3 SW_Push_45deg, SW4 SW_Push_45deg, SW5 SW_Push_45deg, SW6 SW_Push_45deg, SW7 SW_Push_45deg, SW8 SW_Push_45deg, SW9 SW_Push_45deg

Commit message: DecentXE rev 16
[x] Power LED switched to red in BOM
[x] Optional red LED diffuser 3D model
[x] Mid-keyboard support 3D model
[x] Back of the board padding 3D model for better fit in the XE case
[x] Console keys have stabilization holes in PCB and plate
[x] Plate covers the whole width of the keyboard and conoles keys area
[x] PCB made 1.75mm deeper to reach the case's fins on the back of the keyboard area
[x] Remove legends from plate front so it's a uniform black between key caps
Parts:
- D1: JLCPCB Part # C2290 -> C2286
Other:
- company: Decent Consulting -> Decent Engineering
Changed lines of the file:
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@@
 (kicad_sch
-	(version 20231120)
+	(version 20250114)
 	(generator "eeschema")
-	(generator_version "8.0")
+	(generator_version "9.0")
 	(paper "A4")
 	(title_block
 		(title "Decent XE Keyboard - Modern")
-		(date "2024-02-26")
-		(rev "15")
-		(company "Decent Consulting")
+		(date "2026-02-01")
+		(rev "16")
+		(company "Decent Engineering")
+	)
+	(text "Note: columns are high, rows are low."
+		(exclude_from_sim no)
+		(at 78.74 179.07 0)
+		(effects
+			(font
+				(size 1.27 1.27)
+			)
+			(justify left bottom)
+		)
 	)
 	(junction
@@
 		)
 	)
-	(text "Note: columns are high, rows are low."
-		(exclude_from_sim no)
-		(at 78.74 179.07 0)
-		(effects
-			(font
-				(size 1.27 1.27)
-			)
-			(justify left bottom)
-		)
-	)
 	(global_label "COL_4"
 		(shape output)
@@
 			)
 		)
-		(property "JLCPCB Part #" "C2290"
+		(property "JLCPCB Part #" "C2286"
 			(at 229.87 129.54 0)
 			(effects
@@
 		)
 	)
+	(embedded_fonts no)
 )

Commit message: Fabrication tweaks for DecentXE
Parts:
- RV1: JLCPCB Rotation Offset 180 -> (none); Rotation Offset (none) -> 180
- SW0, SW1, SW2, SW3, SW4, SW5, SW6, SW7, SW8, SW9, SWA1, SWB1, SWBrk1, SWC1, SWComma1, SWCps1, SWCtl1, SWD1, SWDash1, SWE1, SWEqual1, SWEsc1, SWF1, SWG1, SWGT1, SWH1, SWI1, SWInv1, SWJ1, SWK1, SWL1, SWLT1, SWM1, SWN1, SWO1, SWP1, SWPeriod1, SWPlus1, SWQ1, SWR1, SWRightSft1, SWS1, SWSemi1, SWSlash1, SWStar1, SWT1, SWTab1, SWU1, SWV1, SWW1, SWX1, SWY1, SWZ1: FT Origin (none) -> Anchor; JLCPCB Position Offset 0,5.5 -> (none); JLCPCB Rotation Offset 180 -> (none); Rotation Offset (none) -> 180
- SWDel1, SWSpc1: FT Origin (none) -> Anchor; JLCPCB Position Offset 0,6 -> (none); JLCPCB Rotation Offset 180 -> (none); Rotation Offset (none) -> 180
- SWFn1, SWFn2, SWFn3, SWFn4, SWHlp1, SWLeftSft1, SWOption1, SWReset1, SWSelect1, SWStart1: FT Origin (none) -> Anchor; JLCPCB Position Offset 0,5.9 -> (none); JLCPCB Rotation Offset 180 -> (none); Rotation Offset (none) -> 180
- SWRet1: FT Origin (none) -> Anchor; JLCPCB Position Offset -2.7,0 -> (none); JLCPCB Rotation Offset 270 -> (none); Rotation Offset (none) -> 270
