File: DecentXE/Keyboard/DecentXE-LowCost.kicad_sch (KiCad schematic)
At the start: 130 parts, among them J1 Conn_02x12_Odd_Even, J2 Conn_01x26, J3 Conn_01x04, SW0 SW_Push_45deg, SW1 SW_Push_45deg, SW2 SW_Push_45deg, SW3 SW_Push_45deg, SW4 SW_Push_45deg, SW5 SW_Push_45deg, SW6 SW_Push_45deg, SW7 SW_Push_45deg, SW8 SW_Push_45deg, SW9 SW_Push_45deg

Commit message: Low-cost version of the DecentXE keyboard
No anti-ghosting
No backlights
No F1-F4 console keys
Only power LED and connector to assemble manually
PCB can be ordered without assembly
Parts:
- removed J1: Conn_02x12_Odd_Even, Connector_IDC:IDC-Header_2x12_P2.54mm_Vertical, symbol Connector_Generic:Conn_02x12_Odd_Even
- added H1, H2: MountingHole, MountingHole:MountingHole_3.2mm_M3, symbol Mechanical:MountingHole
- R1, R10, R11, R12, R13, R14, R15, R16, R17, R18, R19, R2, R20, R21, R22, R23, R24, R25, R26, R27, R28, R29, R3, R30, R31, R32, R33, R34, R35, R36, R37, R38, R39, R4, R40, R41, R42, R43, R44, R45, R46, R47, R48, R49, R50, R51, R52, R53, R54, R55, R57, R59, R6, R60, R61, R62, R63, R64, R65, R66, R8, R9, RV1: now fitted
Connections:
- net ROW_1: now also SWBrk1.2
- net ROW_5: now also SWCtl1.2
- net ROW_8: now also SWLeftSft1.2, SWRightSft1.2
